File: Deckelplatine.sch (EAGLE design)
At the start: 67 parts, among them IC1 MAX1487EESA+, IC2 74HCT595D, IC3 74HCT595D, IC4 74HCT595D, IC5 74HCT595D, IC6 74HCT595D, J1 52808-2570, Q1 BC846BSMD, Q2 BC846BSMD, U1 LM2676S, X1 236-404, X2 233-502

Commit message: Nach 2. Bestellung bei Farnell
Schaltregler Induktion musste nochmals ausgewechselt werden da
die vorherige nur aus USA importierbar wäre.
Parts:
- L1: MF BOURNS -> COILCRAFT; MPN SRR1280-150M -> MSS1278-153MLD; OC_FARNELL 2336471 -> 2288501
Changed lines of the file:
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@@
 <grid distance="0.1" unitdist="inch" unit="inch" style="lines" multiple="1" display="no" altdistance="0.01" altunitdist="inch" altunit="inch"/>
 <layers>
-<layer number="1" name="Top" color="4" fill="1" visible="yes" active="no"/>
-<layer number="2" name="Route2" color="1" fill="3" visible="yes" active="no"/>
-<layer number="3" name="Route3" color="4" fill="3" visible="yes" active="no"/>
-<layer number="4" name="Route4" color="1" fill="4" visible="yes" active="no"/>
-<layer number="5" name="Route5" color="4" fill="4" visible="yes" active="no"/>
-<layer number="6" name="Route6" color="1" fill="8" visible="yes" active="no"/>
-<layer number="7" name="Route7" color="4" fill="8" visible="yes" active="no"/>
-<layer number="8" name="Route8" color="1" fill="2" visible="yes" active="no"/>
-<layer number="9" name="Route9" color="4" fill="2" visible="yes" active="no"/>
-<layer number="10" name="Route10" color="1" fill="7" visible="yes" active="no"/>
-<layer number="11" name="Route11" color="4" fill="7" visible="yes" active="no"/>
-<layer number="12" name="Route12" color="1" fill="5" visible="yes" active="no"/>
-<layer number="13" name="Route13" color="4" fill="5" visible="yes" active="no"/>
-<layer number="14" name="Route14" color="1" fill="6" visible="yes" active="no"/>
-<layer number="15" name="Route15" color="4" fill="6" visible="yes" active="no"/>
-<layer number="16" name="Bottom" color="1" fill="1" visible="yes" active="no"/>
-<layer number="17" name="Pads" color="2" fill="1" visible="yes" active="no"/>
-<layer number="18" name="Vias" color="2" fill="1" visible="yes" active="no"/>
-<layer number="19" name="Unrouted" color="6" fill="1" visible="yes" active="no"/>
-<layer number="20" name="Dimension" color="15" fill="1" visible="yes" active="no"/>
-<layer number="21" name="tPlace" color="16" fill="1" visible="yes" active="no"/>
-<layer number="22" name="bPlace" color="14" fill="1" visible="yes" active="no"/>
-<layer number="23" name="tOrigins" color="15" fill="1" visible="yes" active="no"/>
-<layer number="24" name="bOrigins" color="15" fill="1" visible="yes" active="no"/>
-<layer number="25" name="tNames" color="7" fill="1" visible="yes" active="no"/>
-<layer number="26" name="bNames" color="7" fill="1" visible="yes" active="no"/>
-<layer number="27" name="tValues" color="7" fill="1" visible="yes" active="no"/>
-<layer number="28" name="bValues" color="7" fill="1" visible="yes" active="no"/>
+<layer number="1" name="Top" color="4" fill="1" visible="no" active="no"/>
+<layer number="2" name="Route2" color="1" fill="3" visible="no" active="no"/>
+<layer number="3" name="Route3" color="4" fill="3" visible="no" active="no"/>
+<layer number="4" name="Route4" color="1" fill="4" visible="no" active="no"/>
+<layer number="5" name="Route5" color="4" fill="4" visible="no" active="no"/>
+<layer number="6" name="Route6" color="1" fill="8" visible="no" active="no"/>
+<layer number="7" name="Route7" color="4" fill="8" visible="no" active="no"/>
+<layer number="8" name="Route8" color="1" fill="2" visible="no" active="no"/>
+<layer number="9" name="Route9" color="4" fill="2" visible="no" active="no"/>
+<layer number="10" name="Route10" color="1" fill="7" visible="no" active="no"/>
+<layer number="11" name="Route11" color="4" fill="7" visible="no" active="no"/>
+<layer number="12" name="Route12" color="1" fill="5" visible="no" active="no"/>
+<layer number="13" name="Route13" color="4" fill="5" visible="no" active="no"/>
+<layer number="14" name="Route14" color="1" fill="6" visible="no" active="no"/>
+<layer number="15" name="Route15" color="4" fill="6" visible="no" active="no"/>
+<layer number="16" name="Bottom" color="1" fill="1" visible="no" active="no"/>
+<layer number="17" name="Pads" color="2" fill="1" visible="no" active="no"/>
+<layer number="18" name="Vias" color="2" fill="1" visible="no" active="no"/>
+<layer number="19" name="Unrouted" color="6" fill="1" visible="no" active="no"/>
+<layer number="20" name="Dimension" color="15" fill="1" visible="no" active="no"/>
+<layer number="21" name="tPlace" color="16" fill="1" visible="no" active="no"/>
+<layer number="22" name="bPlace" color="14" fill="1" visible="no" active="no"/>
+<layer number="23" name="tOrigins" color="15" fill="1" visible="no" active="no"/>
+<layer number="24" name="bOrigins" color="15" fill="1" visible="no" active="no"/>
+<layer number="25" name="tNames" color="7" fill="1" visible="no" active="no"/>
+<layer number="26" name="bNames" color="7" fill="1" visible="no" active="no"/>
+<layer number="27" name="tValues" color="7" fill="1" visible="no" active="no"/>
+<layer number="28" name="bValues" color="7" fill="1" visible="no" active="no"/>
 <layer number="29" name="tStop" color="7" fill="3" visible="no" active="no"/>
 <layer number="30" name="bStop" color="7" fill="6" visible="no" active="no"/>
@@
 <layer number="35" name="tGlue" color="7" fill="4" visible="no" active="no"/>
 <layer number="36" name="bGlue" color="7" fill="5" visible="no" active="no"/>
-<layer number="37" name="tTest" color="7" fill="1" visible="yes" active="no"/>
-<layer number="38" name="bTest" color="7" fill="1" visible="yes" active="no"/>
+<layer number="37" name="tTest" color="7" fill="1" visible="no" active="no"/>
+<layer number="38" name="bTest" color="7" fill="1" visible="no" active="no"/>
 <layer number="39" name="tKeepout" color="4" fill="11" visible="no" active="no"/>
 <layer number="40" name="bKeepout" color="1" fill="11" visible="no" active="no"/>
@@
 <layer number="44" name="Drills" color="7" fill="1" visible="no" active="no"/>
 <layer number="45" name="Holes" color="7" fill="1" visible="no" active="no"/>
-<layer number="46" name="Milling" color="3" fill="1" visible="yes" active="no"/>
-<layer number="47" name="Measures" color="7" fill="1" visible="yes" active="no"/>
-<layer number="48" name="Document" color="7" fill="1" visible="yes" active="no"/>
-<layer number="49" name="Reference" color="7" fill="1" visible="yes" active="no"/>
-<layer number="50" name="dxf" color="7" fill="1" visible="yes" active="no"/>
-<layer number="51" name="tDocu" color="6" fill="1" visible="yes" active="no"/>
-<layer number="52" name="bDocu" color="7" fill="1" visible="yes" active="no"/>
-<layer number="53" name="tGND_GNDA" color="7" fill="9" visible="yes" active="no"/>
-<layer number="54" name="bGND_GNDA" color="1" fill="9" visible="yes" active="no"/>
-<layer number="56" name="wert" color="7" fill="1" visible="yes" active="no"/>
+<layer number="46" name="Milling" color="3" fill="1" visible="no" active="no"/>
+<layer number="47" name="Measures" color="7" fill="1" visible="no" active="no"/>
+<layer number="48" name="Document" color="7" fill="1" visible="no" active="no"/>
+<layer number="49" name="Reference" color="7" fill="1" visible="no" active="no"/>
+<layer number="50" name="dxf" color="7" fill="1" visible="no" active="no"/>
+<layer number="51" name="tDocu" color="6" fill="1" visible="no" active="no"/>
+<layer number="52" name="bDocu" color="7" fill="1" visible="no" active="no"/>
+<layer number="53" name="tGND_GNDA" color="7" fill="9" visible="no" active="no"/>
+<layer number="54" name="bGND_GNDA" color="1" fill="9" visible="no" active="no"/>
+<layer number="56" name="wert" color="7" fill="1" visible="no" active="no"/>
 <layer number="90" name="Modules" color="5" fill="1" visible="yes" active="yes"/>
 <layer number="91" name="Nets" color="2" fill="1" visible="yes" active="yes"/>
@@
 </part>
 <part name="L1" library="AcceleratedDesigns_Lib" deviceset="SRR1280-150M" device="">
-<attribute name="MF" value="BOURNS"/>
-<attribute name="MPN" value="SRR1280-150M"/>
-<attribute name="OC_FARNELL" value="2336471"/>
+<attribute name="MF" value="COILCRAFT"/>
+<attribute name="MPN" value="MSS1278-153MLD"/>
+<attribute name="OC_FARNELL" value="2288501"/>
 </part>
 <part name="C2" library="AcceleratedDesigns_Lib" deviceset="GRM21BR61E475MA12L" device="" value="4.7 uF">

Commit message: Datasheet Shift Register
Parts:
- U1: OC_FARNELL 2435897 -> 1564684
Connections:
- net LED_RCK renamed LED_ST_CP
- net LED_SCK renamed LED_SH_CP
- net LED_SER renamed LED_DS
- net REL_RCK renamed REL_ST_CP
- new net REL_DS: JP1.34
- new net REL_SH_CP: JP1.36
- net N$44: now also D2.C; no longer D2.K
- net REL_SCK: no longer JP1.36
- net REL_SER: no longer JP1.34
Other:
- moved on the sheet: D1
Changed lines of the file:
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@@
 <attribute name="MF" value="TEXAS INSTRUMENTS"/>
 <attribute name="MPN" value="LM2676SX-5.0/NOPB"/>
-<attribute name="OC_FARNELL" value="2435897"/>
+<attribute name="OC_FARNELL" value="1564684"/>
 </part>
 <part name="C4" library="AcceleratedDesigns_Lib" deviceset="08053C104KAT2A" device="" value="100.0 nF">
@@
 <attribute name="VALUE" x="101.6" y="193.04" size="1.778" layer="96"/>
 </instance>
-<instance part="D1" gate="G$1" x="68.58" y="233.68" rot="R90">
-<attribute name="OC_FARNELL" x="68.58" y="233.68" size="1.27" layer="96" rot="R90" display="off"/>
-<attribute name="MF" x="68.58" y="233.68" size="1.27" layer="96" display="off"/>
-<attribute name="MPN" x="68.58" y="233.68" size="1.27" layer="96" display="off"/>
+<instance part="D1" gate="G$1" x="68.58" y="233.68" rot="R270">
+<attribute name="OC_FARNELL" x="68.58" y="233.68" size="1.27" layer="96" rot="R270" display="off"/>
+<attribute name="MF" x="68.58" y="233.68" size="1.27" layer="96" rot="R180" display="off"/>
+<attribute name="MPN" x="68.58" y="233.68" size="1.27" layer="96" rot="R180" display="off"/>
 </instance>
 <instance part="R4" gate="G$1" x="91.44" y="172.72" smashed="yes">
@@
 </segment>
 </net>
-<net name="LED_SER" class="0">
+<net name="LED_DS" class="0">
 <segment>
 <pinref part="IC4" gate="A" pin="SER"/>
@@
 </segment>
 </net>
-<net name="LED_SCK" class="0">
+<net name="LED_SH_CP" class="0">
 <segment>
 <pinref part="IC4" gate="A" pin="SCK"/>
@@
 </segment>
 </net>
-<net name="LED_RCK" class="0">
+<net name="LED_ST_CP" class="0">
 <segment>
 <pinref part="IC4" gate="A" pin="RCK"/>
@@
 </segment>
 </net>
-<net name="REL_RCK" class="0">
+<net name="REL_ST_CP" class="0">
 <segment>
 <pinref part="IC2" gate="A" pin="RCK"/>
@@
 <label x="266.7" y="71.12" size="1.27" layer="95" rot="R180" xref="yes"/>
 </segment>
-<segment>
-<pinref part="JP1" gate="A" pin="36"/>
-<wire x1="40.64" y1="63.5" x2="48.26" y2="63.5" width="0.1524" layer="91"/>
-<label x="48.26" y="63.5" size="1.27" layer="95" xref="yes"/>
-</segment>
 </net>
 <net name="REL_SER" class="0">
@@
 <wire x1="269.24" y1="111.76" x2="266.7" y2="111.76" width="0.1524" layer="91"/>
 <label x="266.7" y="111.76" size="1.27" layer="95" rot="R180" xref="yes"/>
-</segment>
-<segment>
-<wire x1="40.64" y1="66.04" x2="48.26" y2="66.04" width="0.1524" layer="91"/>
-<pinref part="JP1" gate="A" pin="34"/>
-<label x="48.26" y="66.04" size="1.27" layer="95" xref="yes"/>
 </segment>
 </net>
@@
 </net>
 <net name="12V_VIN" class="0">
-<segment>
-<pinref part="D1" gate="G$1" pin="C"/>
-<wire x1="66.04" y1="233.68" x2="58.42" y2="233.68" width="0.1524" layer="91"/>
-<label x="58.42" y="233.68" size="1.27" layer="95" rot="R180" xref="yes"/>
-</segment>
 <segment>
 <pinref part="X1" gate="G$1" pin="P2.2"/>
@@
 <pinref part="R5" gate="G$1" pin="2"/>
 <wire x1="83.82" y1="210.82" x2="81.28" y2="210.82" width="0.1524" layer="91"/>
+<pinref part="D1" gate="G$1" pin="C"/>
+<wire x1="71.12" y1="233.68" x2="81.28" y2="233.68" width="0.1524" layer="91"/>
+<junction x="81.28" y="233.68"/>
+</segment>
+<segment>
 <pinref part="D1" gate="G$1" pin="A"/>
-<wire x1="81.28" y1="233.68" x2="71.12" y2="233.68" width="0.1524" layer="91"/>
-<junction x="81.28" y="233.68"/>
+<wire x1="66.04" y1="233.68" x2="58.42" y2="233.68" width="0.1524" layer="91"/>
+<label x="58.42" y="233.68" size="1.27" layer="95" rot="R180" xref="yes"/>
 </segment>
 </net>
@@
 <junction x="205.74" y="233.68"/>
 <junction x="205.74" y="228.6"/>
-<pinref part="D2" gate="A" pin="K"/>
+<pinref part="D2" gate="A" pin="C"/>
 <wire x1="205.74" y1="218.79" x2="205.74" y2="228.6" width="0.1524" layer="91"/>
 </segment>
@@
 </segment>
 </net>
+<net name="REL_DS" class="0">
+<segment>
+<wire x1="40.64" y1="66.04" x2="48.26" y2="66.04" width="0.1524" layer="91"/>
+<pinref part="JP1" gate="A" pin="34"/>
+<label x="48.26" y="66.04" size="1.27" layer="95" xref="yes"/>
+</segment>
+</net>
+<net name="REL_SH_CP" class="0">
+<segment>
+<pinref part="JP1" gate="A" pin="36"/>
+<wire x1="40.64" y1="63.5" x2="48.26" y2="63.5" width="0.1524" layer="91"/>
+<label x="48.26" y="63.5" size="1.27" layer="95" xref="yes"/>
+</segment>
+</net>

Commit message: Zwischen Commit Änderungen leider nicht mehr klar
Leider habe ich vergessen welche Änderungen dieser Commit mit sich brachte.
Desshalb sollte dieser komplett ignoriert werden.
Parts:
- C10, C11, C7, C8, C9: value 100n -> 0.1uF
- C4: value 100.0 nF -> 0.1uF
- X1: value 236-404 -> 236-406/000-023; device con-wago_236:236-404 -> con-wago_236:236-406/000-023; MPN 236-404 -> 236-406; OC_FARNELL 1283528 -> 1283529
Connections:
- removed net REL_SCK: IC2A.SCK, IC3A.SCK
- removed net REL_SER: IC2A.SER
- new net LED_!OE: IC4A.G, IC5A.G, IC6A.G, JP1.31
- new net REL_!OE: IC2A.G, IC3A.G, JP1.32
- net 12V_VIN: now also X1.P4.1, X1.P4.2
- net ACCU+: now also X1.P6.1, X1.P6.2; no longer X1.P4.1, X1.P4.2
- net GND: now also X1.P5.1, X1.P5.2; no longer IC2A.G, IC3A.G, IC4A.G, IC5A.G, IC6A.G
- net REL_DS: now also IC2A.SER
- net REL_SH_CP: now also IC2A.SCK, IC3A.SCK
Other:
- note added: "ACHTUNG!!! Connector erscheint gedreht im Vergleich zur PIN Belegung des Banana Pro!"
- note added: "Boden+"
- note added: "Boden-"
- note added: "Deckel+"
- note added: "Deckel-"
- note removed: "ACHTUNG! Connector erscheint gedreht im Vergleich zur PIN Belegung des Banana Pro!"
- moved on the sheet: D1, H1, H2, H3, H4, TP1, TP2, X2
