File: Deckelplatine.sch (EAGLE design)
At the start: 59 parts, among them IC1 MAX1487EESA+, IC2 74HCT595D, IC3 74HCT595D, IC4 74HCT595D, IC5 74HCT595D, IC6 74HCT595D, J1 52808-2570, U1 LM2676S, X1 236-406/000-023, X2 233-502

Commit message: Ein wenig Kosmetik auf der Deckelplatine
Beschriftungen angepasst
Parts:
- F1: value 0.63AT -> 2AT
Changed lines of the file:
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@@
 <attribute name="OC_FARNELL" value="unknown"/>
 </part>
-<part name="F1" library="fuse-littlefuse" deviceset="01110005MR" device="" value="0.63AT">
+<part name="F1" library="fuse-littlefuse" deviceset="01110005MR" device="" value="2AT">
 <attribute name="MF" value="LITTELFUSE"/>
 <attribute name="MPN" value="01110005MR"/>
@@
 <pinref part="U1" gate="G$1" pin="IN"/>
 <wire x1="76.2" y1="233.68" x2="81.28" y2="233.68" width="0.1524" layer="91"/>
-<wire x1="81.28" y1="233.68" x2="124.46" y2="233.68" width="0.1524" layer="91"/>
-<wire x1="124.46" y1="233.68" x2="137.16" y2="233.68" width="0.1524" layer="91"/>
+<wire x1="81.28" y1="233.68" x2="91.44" y2="233.68" width="0.1524" layer="91"/>
+<wire x1="91.44" y1="233.68" x2="137.16" y2="233.68" width="0.1524" layer="91"/>
 <wire x1="154.94" y1="233.68" x2="152.4" y2="233.68" width="0.1524" layer="91"/>
 <pinref part="C4" gate="A" pin="1"/>
@@
 <junction x="137.16" y="228.6"/>
 <junction x="137.16" y="233.68"/>
-<wire x1="124.46" y1="180.34" x2="81.28" y2="180.34" width="0.1524" layer="91"/>
-<wire x1="124.46" y1="180.34" x2="124.46" y2="233.68" width="0.1524" layer="91"/>
-<junction x="124.46" y="233.68"/>
+<wire x1="91.44" y1="180.34" x2="81.28" y2="180.34" width="0.1524" layer="91"/>
+<wire x1="91.44" y1="180.34" x2="91.44" y2="233.68" width="0.1524" layer="91"/>
+<junction x="91.44" y="233.68"/>
 <pinref part="F2" gate="G$1" pin="2A"/>
 <pinref part="D1" gate="G$1" pin="C"/>
