File: Bodenplatine v001.brd (EAGLE design)
At the start: 290 x 145 mm, 113 parts, among them K1 RY612012, K2 RY612012, K3 RY612012, K4 RY612012, K5 RY612012, K6 RY612012, K7 RY612012, K8 RY612012, K9 RY612012, Q1 BC846BLT1SMD, Q2 BC846BLT1SMD, Q3 BC846BLT1SMD, Q4 BC846BLT1SMD, Q5 BC846BLT1SMD, Q6 BC846BLT1SMD, Q7 BC846BLT1SMD, Q8 BC846BLT1SMD, Q9 BC846BLT1SMD, X1 SPRINGCON_AST125_5X2, X10 SPRINGCON_AST125_3X2, X11 SPRINGCON_AST125_4X2, X12 SPRINGCON_AST125_4X2, X13 SPRINGCON_AST125_5X2, X14 236-403, X15 236-402, X2 SPRINGCON_AST125_5X2, X3 SPRINGCON_AST125_5X2, X4 SPRINGCON_AST125_5X2, X5 SPRINGCON_AST125_5X2, X6 SPRINGCON_AST125_5X2, X7 SPRINGCON_AST125_5X2, X8 SPRINGCON_AST125_5X2, X9 SPRINGCON_AST125_5X2

Commit message: Alle Bauteile auf dem Board, teilweise genau positioniert.
GND ground plane auf beiden Seiten
Parts:
- moved R24 316.1 mm to (273.0, 113.5)
- moved D16 316.0 mm to (274.1, 121.4)
- moved R20 311.2 mm to (271.1, 105.0)
- moved D26 307.8 mm to (264.1, 104.7), turned to 90 degrees
- moved D15 296.4 mm to (246.4, 121.9)
- moved R19 292.5 mm to (241.9, 106.0)
- moved R16 274.9 mm to (271.9, 127.8)
- moved D20 262.2 mm to (236.8, 105.6), turned to 90 degrees
- moved R15 255.8 mm to (246.0, 127.8)
- moved R12 248.6 mm to (160.0, 115.6)
- moved D19 238.7 mm to (208.3, 105.3), turned to 90 degrees
- moved R14 232.2 mm to (215.2, 126.8)
- moved D4 220.0 mm to (160.8, 121.6)
- moved D18 214.5 mm to (178.8, 105.0), turned to 90 degrees
- moved R4 213.7 mm to (159.8, 127.4)
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Routing:
- added copper zone on layer 1, net N$93
- added copper zone on layer 16, net N$95
Other:
- board text added: "Relais 1"
- board text added: "Relais 2"
- board text added: "Relais 3"
- board text added: "Relais 4"
- board text added: "Relais 5"
- board text added: "Relais 6"
- board text added: "Relais 7"
- board text added: "Relais 8"
- board text added: "Relais 9"
