File: Bodenplatine v001.brd (EAGLE design)
At the start: 290 x 145 mm, 113 parts, among them K1 RY612012, K2 RY612012, K3 RY612012, K4 RY612012, K5 RY612012, K6 RY612012, K7 RY612012, K8 RY612012, K9 RY612012, Q1 BC846BLT1SMD, Q2 BC846BLT1SMD, Q3 BC846BLT1SMD, Q4 BC846BLT1SMD, Q5 BC846BLT1SMD, Q6 BC846BLT1SMD, Q7 BC846BLT1SMD, Q8 BC846BLT1SMD, Q9 BC846BLT1SMD, X1 SPRINGCON_AST125_5X2, X10 SPRINGCON_AST125_3X2, X11 SPRINGCON_AST125_4X2, X12 SPRINGCON_AST125_4X2, X13 SPRINGCON_AST125_5X2, X14 236-403, X15 236-402, X2 SPRINGCON_AST125_5X2, X3 SPRINGCON_AST125_5X2, X4 SPRINGCON_AST125_5X2, X5 SPRINGCON_AST125_5X2, X6 SPRINGCON_AST125_5X2, X7 SPRINGCON_AST125_5X2, X8 SPRINGCON_AST125_5X2, X9 SPRINGCON_AST125_5X2

Commit message: Leucht Dioden ausgerichtet
Parts:
- moved D7 2.54 mm to (92.5, 105.0)
- moved D5 2.48 mm to (35.0, 105.0)
- moved D6 2.44 mm to (63.8, 105.0)
- moved D8 1.99 mm to (121.2, 105.0)
- moved D17 1.97 mm to (150.0, 105.0)
- moved D19 1.74 mm to (207.5, 105.0)
- moved D26 1.27 mm to (265.0, 105.0), turned to 90 degrees
- moved D18 1.26 mm to (178.8, 105.0)
- moved D20 0.80 mm to (236.2, 105.0)

Commit message: NPN Transistoren ausgerichtet
Parts:
- moved D3 1.86 mm to (126.2, 117.0)
- moved D4 1.69 mm to (155.0, 117.0)
- moved D13 1.47 mm to (183.8, 117.0)
- moved D15 1.30 mm to (241.2, 117.0)
- moved D2 1.17 mm to (97.5, 117.0)
- moved D14 1.14 mm to (212.5, 117.0)
- moved D16 1.08 mm to (270.0, 117.0)
- moved D1 0.62 mm to (68.8, 117.0)
- moved R2 0.54 mm to (102.8, 117.0)
- moved R1 0.53 mm to (74.0, 117.0)
- moved R15 0.50 mm to (246.8, 117.0)
- moved R25 0.46 mm to (45.9, 117.0)
- moved D25 0.43 mm to (40.0, 117.0)
- moved R14 0.40 mm to (217.3, 117.0)
- moved R4 0.37 mm to (160.9, 117.0)
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Routing:
- net N$78: track 0.00 -> 12.4 mm
- net N$28: track 0.00 -> 12.3 mm
- net N$18: track 0.00 -> 12.0 mm
- net N$68: track 0.00 -> 11.6 mm
- net N$5: track 0.00 -> 10.9 mm
- net N$58: track 0.00 -> 10.5 mm
- net N$48: track 0.00 -> 10.3 mm
- net N$38: track 0.00 -> 10.3 mm
- net N$88: track 0.00 -> 9.67 mm
- net N$77: track 0.00 -> 5.17 mm
- net N$67: track 0.00 -> 5.17 mm
- net N$57: track 0.00 -> 5.17 mm
- net N$47: track 0.00 -> 5.17 mm
- net N$37: track 0.00 -> 5.17 mm
- net N$27: track 0.00 -> 5.17 mm
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
Commit message: Vertauschte Dioden gefixt
Parts:
- removed D17, D18, D19, D20, D26: Yellow, SparkFun-LED:LED-0603
- removed F13: 3,15AT, xMZ-Mod-Touch-Bodenplatine:FPG4
- added F11: 3,15AT, xMZ-Mod-Touch-Bodenplatine:FPG4
- added V2, V3, V4, V9: BAR43, xMZ-Mod-Touch-Bodenplatine:SOT323
- added V6: 1N4148W, xMZ-Mod-Touch-Bodenplatine:MINIMELF
- D1, D2, D3, D4: value BAR43 -> Yellow; device xMZ-Mod-Touch-Bodenplatine:SOT323 -> SparkFun-LED:LED-0603
- D9: value 1N4148W -> Yellow; device xMZ-Mod-Touch-Bodenplatine:MINIMELF -> SparkFun-LED:LED-0603
- F10: value 10AT -> 6,3AT
- F12: value 6,3AT -> 3,15AT
- F9: value 3,15AT -> 10AT
- X10: value SPRINGCON_AST125_3X2 -> SPRINGCON_AST125_4X2; device xMZ-Mod-Touch-Bodenplatine:SPRINGCON_AST125_3X2 -> xMZ-Mod-Touch-Bodenplatine:SPRINGCON_AST125_4X2
- X11: value SPRINGCON_AST125_4X2 -> SPRINGCON_AST125_5X2; device xMZ-Mod-Touch-Bodenplatine:SPRINGCON_AST125_4X2 -> xMZ-Mod-Touch-Bodenplatine:SPRINGCON_AST125_5X2
- X12: value SPRINGCON_AST125_4X2 -> 236-403; device xMZ-Mod-Touch-Bodenplatine:SPRINGCON_AST125_4X2 -> con-wago_236:P-236-403
- X13: value SPRINGCON_AST125_5X2 -> 236-402; device xMZ-Mod-Touch-Bodenplatine:SPRINGCON_AST125_5X2 -> con-wago_236:P-236-402
- X14: value 236-403 -> SPRINGCON_AST125_4X2; device con-wago_236:P-236-403 -> xMZ-Mod-Touch-Bodenplatine:SPRINGCON_AST125_4X2
- X15: value 236-402 -> SPRINGCON_AST125_5X2; device con-wago_236:P-236-402 -> xMZ-Mod-Touch-Bodenplatine:SPRINGCON_AST125_5X2
- X9: value SPRINGCON_AST125_5X2 -> SPRINGCON_AST125_3X2; device xMZ-Mod-Touch-Bodenplatine:SPRINGCON_AST125_5X2 -> xMZ-Mod-Touch-Bodenplatine:SPRINGCON_AST125_3X2
- moved F9 234.0 mm to (23.0, 23.0), turned to 0 degrees
- moved R27 230.2 mm to (270.5, 109.7)
- moved R26 229.8 mm to (269.9, 113.5), turned to 0 degrees
- moved R25 228.8 mm to (274.8, 117.0)
- moved X9 217.4 mm to (45.0, 18.0)
- moved X13 217.0 mm to (53.0, 128.0), turned to 90 degrees
- moved X15 217.0 mm to (240.0, 18.0), turned to 0 degrees
- moved D9 201.3 mm to (265.0, 105.0), turned to 90 degrees
- moved X12 193.4 mm to (12.0, 129.5), turned to 90 degrees
- moved X14 193.4 mm to (170.0, 18.0), turned to 0 degrees
- moved X11 143.6 mm to (260.0, 50.0)
- moved F10 122.0 mm to (145.0, 23.0)
- moved D5 115.0 mm to (150.0, 105.0)
- moved D6 115.0 mm to (178.8, 105.0)
- moved D7 115.0 mm to (207.5, 105.0)
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- renumbered D10 to V7, D11 to V8, D12 to V13, D13 to V10, D14 to V11, D15 to V12, D16 to V17, D21 to V14, D22 to V15, D23 to V16, D24 to V18, D25 to V1, D27 to V5
Connections:
- net 12V: now also F10.1, F10.1', X13.L1.1, X13.L1.2; no longer F13.1, F13.1', X15.L1.1, X15.L1.2
- net A-: now also X15.4, X15.4'; no longer X13.4, X13.4'
- net B+: now also X15.3, X15.3'; no longer X13.3, X13.3'
- net GND: now also D1.C, D2.C, D3.C, D4.C, D9.C, X13.L2.1, X13.L2.2, X14.3, X14.3', X14.4, X14.4', X15.2, X15.2'; no longer D17.C, D18.C, D19.C, D20.C, D26.C, X12.3, X12.3', X12.4, X12.4', X13.2, X13.2', X15.L2.1, X15.L2.2
- net L: now also F9.1, F9.1', X10.1, X10.1', X10.2, X10.2', X10.3, X10.3', X10.4, X10.4', X12.L1.1, X12.L1.2; no longer F10.1, F10.1', X11.1, X11.1', X11.2, X11.2', X11.3, X11.3', X11.4, X11.4', X14.L1.1, X14.L1.2
- net N: now also X11.4, X11.4', X12.L2.1, X12.L2.2, X9.2, X9.2'; no longer X10.2, X10.2', X14.L2.1, X14.L2.2, X9.4, X9.4'
- net N$1: now also X3.2, X3.2'; no longer X2.2, X2.2'
- net N$10: now also R10.2; no longer R9.2
- net N$11: now also V6.C; no longer D9.C
- net N$13: now also R3.1, V3.1; no longer D2.1, R2.1
- net N$14: now also R11.1, R7.2, V3.3; no longer D2.3, R10.1, R6.2
- net N$15: now also D3.A, R7.1; no longer D6.A, R6.1
- net N$16: now also R11.2; no longer R10.2
- net N$19: now also X2.2, X2.2'; no longer X3.2, X3.2'
- net N$2: now also X3.3, X3.3'; no longer X2.3, X2.3'
- net N$20: now also X2.1, X2.1'; no longer X3.1, X3.1'
- net N$23: now also R4.1, V4.1; no longer D3.1, R3.1
- net N$24: now also R12.1, R8.2, V4.3; no longer D3.3, R11.1, R7.2
- net N$25: now also D4.A, R8.1; no longer D7.A, R7.1
- net N$26: now also R12.2; no longer R11.2
- net N$33: now also R13.1, V9.1; no longer D4.1, R4.1
- net N$34: now also R17.2, R21.1, V9.3; no longer D4.3, R12.1, R8.2
- net N$35: now also D5.A, R17.1; no longer D8.A, R8.1
- net N$36: now also R21.2; no longer R12.2
- net N$4: now also X3.1, X3.1'; no longer X2.1, X2.1'
- net N$43: now also R14.1; no longer R13.1
- net N$44: now also R18.2, R22.1; no longer R17.2, R21.1
- net N$45: now also D6.A, R18.1; no longer D17.A, R17.1
- net N$46: now also R22.2; no longer R21.2
- net N$5: now also V6.A; no longer D9.A
- net N$53: now also R15.1; no longer R14.1
- net N$54: now also R19.2, R23.1; no longer R18.2, R22.1
- net N$55: now also D7.A, R19.1; no longer D18.A, R18.1
- net N$56: now also R23.2; no longer R22.2
- net N$6: now also X2.3, X2.3'; no longer X3.3, X3.3'
- net N$63: now also R16.1; no longer R15.1
- net N$64: now also R20.2, R24.1; no longer R19.2, R23.1
- net N$65: now also D8.A, R20.1; no longer D19.A, R19.1
- net N$66: now also R24.2; no longer R23.2
- net N$7: now also R2.1, V2.1; no longer D1.1, R1.1
- net N$71: now also X11.3, X11.3'; no longer X9.3, X9.3'
- net N$72: now also F11.2, F11.2'; no longer F9.2, F9.2'
- net N$73: now also R25.1; no longer R16.1
- net N$74: now also R26.2, R27.1; no longer R20.2, R24.1
- net N$75: now also D9.A, R26.1; no longer D20.A, R20.1
- net N$76: now also R27.2; no longer R24.2
- net N$79: now also F11.1, F11.1', X11.2, X11.2'; no longer F9.1, F9.1', X9.2, X9.2'
- net N$8: now also R10.1, R6.2, V2.3; no longer D1.3, R5.2, R9.1
- net N$80: now also X11.1, X11.1'; no longer X9.1, X9.1'
- net N$83: now also R1.1; no longer R25.1
- net N$84: now also R5.2, R9.1; no longer R26.2, R27.1
- net N$85: now also D1.A, R5.1; no longer D26.A, R26.1
- net N$86: now also R9.2; no longer R27.2
- net N$9: now also D2.A, R6.1; no longer D5.A, R5.1
- net N$91: now also F9.2, F9.2', X9.1, X9.1'; no longer F10.2, F10.2', X10.1, X10.1'
- net N$92: now also F12.2, F12.2', X15.1, X15.1'; no longer F13.2, F13.2', X13.1, X13.1'
- net N$94: now also F10.2, F10.2', X14.1, X14.1', X14.2, X14.2'; no longer F12.2, F12.2', X12.1, X12.1', X12.2, X12.2'
- net P1: now also R1.2; no longer R25.2
- net P2: now also R2.2; no longer R1.2
- net P3: now also R3.2; no longer R2.2
- net P4: now also R4.2; no longer R3.2
- net P5: now also R13.2; no longer R4.2
- net P6: now also R14.2; no longer R13.2
- net P7: now also R15.2; no longer R14.2
- net P8: now also R16.2; no longer R15.2
- net P9: now also R25.2; no longer R16.2
- net PE: now also X11.5, X11.5', X12.L3.1, X12.L3.2, X9.3, X9.3'; no longer X10.3, X10.3', X14.L3.1, X14.L3.2, X9.5, X9.5'
- net SCHIRM: now also X15.5, X15.5'; no longer X13.5, X13.5'

Commit message: Widerstände und Dioden ausgerichtet
Parts:
- moved R5 5.49 mm to (37.0, 110.0), turned to 0 degrees
- moved R6 4.75 mm to (65.8, 110.0), turned to 0 degrees
- moved R7 4.56 mm to (94.5, 110.0), turned to 0 degrees
- moved R26 4.54 mm to (267.0, 110.0)
- moved R8 3.93 mm to (123.2, 110.0)
- moved R17 3.89 mm to (152.0, 110.0)
- moved R19 3.85 mm to (209.5, 110.0)
- moved R18 3.70 mm to (180.8, 110.0)
- moved R20 3.35 mm to (238.2, 110.0)
- moved Q9 3.21 mm to (271.0, 105.0)
- moved Q4 3.17 mm to (127.2, 105.0)
- moved Q8 2.64 mm to (242.2, 105.0)
- moved Q7 2.59 mm to (213.5, 105.0)
- moved Q6 2.16 mm to (184.8, 105.0)
- moved Q3 1.93 mm to (98.5, 105.0)
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Routing:
- net N$78: track 12.4 -> 0.00 mm
- net N$28: track 12.3 -> 0.00 mm
- net N$68: track 11.6 -> 0.00 mm
- net N$58: track 10.5 -> 0.00 mm
- net N$48: track 10.3 -> 0.00 mm
- net N$18: track 12.0 -> 5.17 mm
- net N$5: track 10.9 -> 5.17 mm
- net N$38: track 10.3 -> 5.17 mm
- net N$88: track 9.67 -> 5.17 mm

Commit message: Begin Änderungen der Klemmenbezeichnungen
Parts:
- removed X10: SPRINGCON_AST125_4X2, xMZ-Mod-Touch-Bodenplatine:SPRINGCON_AST125_4X2
- removed X12: 236-403, con-wago_236:P-236-403
- removed X2: SPRINGCON_AST125_5X2, xMZ-Mod-Touch-Bodenplatine:SPRINGCON_AST125_5X2
- added X12.: SPRINGCON_AST125_4X2, xMZ-Mod-Touch-Bodenplatine:SPRINGCON_AST125_4X2
- added X2., X9.: SPRINGCON_AST125_5X2, xMZ-Mod-Touch-Bodenplatine:SPRINGCON_AST125_5X2
- X11: value SPRINGCON_AST125_5X2 -> SPRINGCON_AST125_4X2; device xMZ-Mod-Touch-Bodenplatine:SPRINGCON_AST125_5X2 -> xMZ-Mod-Touch-Bodenplatine:SPRINGCON_AST125_4X2
- X14: value SPRINGCON_AST125_4X2 -> 236-403; device xMZ-Mod-Touch-Bodenplatine:SPRINGCON_AST125_4X2 -> con-wago_236:P-236-403
- moved X14 193.4 mm to (12.0, 129.5), turned to 90 degrees
- moved X11 143.6 mm to (120.0, 18.0)
- moved X3 28.8 mm to (87.5, 50.0)
- moved R1 0.92 mm to (45.0, 117.0)
- moved R4 0.91 mm to (131.2, 117.0)
- moved R13 0.87 mm to (160.0, 117.0)
- moved R16 0.58 mm to (246.2, 117.0)
- moved R2 0.26 mm to (73.8, 117.0)
- moved R3 0.25 mm to (102.5, 117.0)
- moved R25 0.23 mm to (275.0, 117.0)
- moved R15 0.15 mm to (217.5, 117.0)
- moved R14 0.11 mm to (188.8, 117.0)
- renumbered X15 to X13., X9 to X10.
Connections:
- net GND: now also X12..3, X12..3', X12..4, X12..4'; no longer X14.3, X14.3', X14.4, X14.4'
- net L: now also X11.1, X11.1', X11.2, X11.2', X11.3, X11.3', X11.4, X11.4', X14.L1.1, X14.L1.2; no longer X10.1, X10.1', X10.2, X10.2', X10.3, X10.3', X10.4, X10.4', X12.L1.1, X12.L1.2
- net N: now also X14.L2.1, X14.L2.2, X2..4, X2..4', X9..4, X9..4'; no longer X11.4, X11.4', X12.L2.1, X12.L2.2, X2.4, X2.4'
- net N$1: now also X2..2, X2..2'; no longer X3.2, X3.2'
- net N$19: now also X3.2, X3.2'; no longer X2.2, X2.2'
- net N$2: now also X2..3, X2..3'; no longer X3.3, X3.3'
- net N$20: now also X3.1, X3.1'; no longer X2.1, X2.1'
- net N$4: now also X2..1, X2..1'; no longer X3.1, X3.1'
- net N$6: now also X3.3, X3.3'; no longer X2.3, X2.3'
- net N$71: now also X9..3, X9..3'; no longer X11.3, X11.3'
- net N$79: now also X9..2, X9..2'; no longer X11.2, X11.2'
- net N$80: now also X9..1, X9..1'; no longer X11.1, X11.1'
- net N$94: now also X12..1, X12..1', X12..2, X12..2'; no longer X14.1, X14.1', X14.2, X14.2'
- net PE: now also X14.L3.1, X14.L3.2, X2..5, X2..5', X9..5, X9..5'; no longer X11.5, X11.5', X12.L3.1, X12.L3.2, X2.5, X2.5'
Routing:
- net P9: track 0.00 -> 131.3 mm
- net P1: track 0.00 -> 105.2 mm
- net P8: track 0.00 -> 105.1 mm
- net P7: track 0.00 -> 78.9 mm
- net P2: track 0.00 -> 73.8 mm
- net P6: track 0.00 -> 60.0 mm
- net P3: track 0.00 -> 39.3 mm
- net P5: track 0.00 -> 33.8 mm
- net 5V: track 230.0 -> 248.2 mm
- net P4: track 0.00 -> 17.1 mm
- net N$14: track 0.00 -> 13.9 mm
- net N$64: track 0.00 -> 13.9 mm
- net N$44: track 0.00 -> 13.8 mm
- net N$74: track 0.00 -> 13.8 mm
- net N$34: track 0.00 -> 13.8 mm
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
Commit message: Erste finale Version OHNE CHECKS
Parts:
- removed F11: 3,15AT, xMZ-Mod-Touch-Bodenplatine:FPG4
- removed X13.: SPRINGCON_AST125_5X2, xMZ-Mod-Touch-Bodenplatine:SPRINGCON_AST125_5X2
- added F13: 3,15AT, xMZ-Mod-Touch-Bodenplatine:FPG4
- added X15: 236-402, xMZ-Mod-Touch-Bodenplatine:P-236-402
- F10: value 6,3AT -> 10AT
- F12: value 3,15AT -> 6,3AT
- F9: value 10AT -> 3,15AT
- X13: value 236-402 -> SPRINGCON_AST125_5X2; device con-wago_236:P-236-402 -> xMZ-Mod-Touch-Bodenplatine:SPRINGCON_AST125_5X2
- X14: device con-wago_236:P-236-403 -> xMZ-Mod-Touch-Bodenplatine:P-236-403
- moved F9 234.0 mm to (251.0, 75.5), turned to 90 degrees
- moved X13 217.0 mm to (240.0, 18.0), turned to 0 degrees
- moved F10 122.0 mm to (23.0, 23.0)
- moved F12 75.0 mm to (145.0, 23.0)
- renumbered X10. to X10, X12. to X12, X2. to X2, X9. to X9
Connections:
- net 12V: now also F13.1, F13.1', X15.L1.1, X15.L1.2; no longer F10.1, F10.1', X13.L1.1, X13.L1.2
- net A-: now also X13.4, X13.4'; no longer X13..4, X13..4'
- net B+: now also X13.3, X13.3'; no longer X13..3, X13..3'
- net GND: now also X13.2, X13.2', X15.L2.1, X15.L2.2; no longer X13..2, X13..2', X13.L2.1, X13.L2.2
- net L: now also F10.1, F10.1'; no longer F9.1, F9.1'
- net N$72: now also F9.2, F9.2'; no longer F11.2, F11.2'
- net N$79: now also F9.1, F9.1'; no longer F11.1, F11.1'
- net N$91: now also F10.2, F10.2'; no longer F9.2, F9.2'
- net N$92: now also F13.2, F13.2', X13.1, X13.1'; no longer F12.2, F12.2', X13..1, X13..1'
- net N$94: now also F12.2, F12.2'; no longer F10.2, F10.2'
- net SCHIRM: now also X13.5, X13.5'; no longer X13..5, X13..5'
Routing:
- net 12V: track 489.3 -> 502.7 mm, vias 3 -> 0

Commit message: Alle Datasheets der Bodenplatine vorhanden
Auserdem noch einige Änderungen an den Footprints der Bodenplatine
Parts:
- D1, D2, D3, D4, D5, D6, D7, D8, D9: value Yellow -> YELLOW; device SparkFun-LED:LED-0603 -> xMZ-Mod-Touch-Bodenplatine:LED-1206
- V1, V10, V11, V12, V17, V2, V3, V4, V9: value BAR43 -> BAR43SOT233; device xMZ-Mod-Touch-Bodenplatine:SOT323 -> xMZ-Mod-Touch-Bodenplatine:SOT23
- turned D1 to 180 degrees
- turned D2 to 180 degrees
- turned D3 to 180 degrees
- turned D4 to 180 degrees
- turned D5 to 180 degrees
- turned D6 to 180 degrees
- turned D7 to 180 degrees
- turned D8 to 180 degrees
- turned D9 to 180 degrees
Routing:
- net GND: track 361.9 -> 20.2 mm, vias 1 -> 0
- net N: track 367.4 -> 372.9 mm
- net PE: track 378.7 -> 376.4 mm
- net A-: track 269.7 -> 271.9 mm
- net B+: track 267.1 -> 269.2 mm

Commit message: Logos auf dem Board und Außenmaße mit Kerben
Parts:
- added U$1: (no value), xMZ-Mod-Touch-Bodenplatine:TEXT_FUSE
- added U$2: (no value), xMZ-Mod-Touch-Bodenplatine:TEXT_NAME_VERSION_AUTHOR
- added U$3: (no value), xMZ-Mod-Touch-Bodenplatine:LOGO_RA-GAS
- added U$4, U$5: (no value), xMZ-Mod-Touch-Bodenplatine:LOGO_RA-GAS_BOTTOM
Other:
- outline, holes or cut-outs redrawn
- board text added: "COM"
- board text added: "NC"
- board text added: "NO"
- board text removed: ">AUTHOR"
- board text removed: ">PROJEKTNAME"
- board text removed: ">VERSION"
- board text removed: "v"
Changed lines of the file:
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@@
 <setting verticaltext="up"/>
 </settings>
-<grid distance="0.05" unitdist="inch" unit="inch" style="lines" multiple="1" display="yes" altdistance="0.005" altunitdist="inch" altunit="inch"/>
+<grid distance="0.5" unitdist="mm" unit="mm" style="lines" multiple="1" display="yes" altdistance="0.1" altunitdist="mm" altunit="mm"/>
 <layers>
 <layer number="1" name="Top" color="4" fill="1" visible="yes" active="yes"/>
@@
 <layer number="23" name="tOrigins" color="15" fill="1" visible="yes" active="yes"/>
 <layer number="24" name="bOrigins" color="15" fill="1" visible="yes" active="yes"/>
-<layer number="25" name="tNames" color="7" fill="1" visible="no" active="yes"/>
+<layer number="25" name="tNames" color="7" fill="1" visible="yes" active="yes"/>
 <layer number="26" name="bNames" color="7" fill="1" visible="no" active="yes"/>
 <layer number="27" name="tValues" color="7" fill="1" visible="no" active="yes"/>
@@
 <plain>
 <wire x1="0" y1="0" x2="290" y2="0" width="0" layer="20"/>
-<wire x1="290" y1="0" x2="290" y2="145" width="0" layer="20"/>
 <wire x1="290" y1="145" x2="0" y2="145" width="0" layer="20"/>
-<wire x1="0" y1="145" x2="0" y2="0" width="0" layer="20"/>
 <text x="28.5" y="85" size="1.778" layer="21" font="vector" ratio="15" rot="R90">Relais 1</text>
 <text x="57.5" y="85" size="1.778" layer="21" font="vector" ratio="15" rot="R90">Relais 2</text>
@@
 <text x="59" y="11" size="1.778" layer="21" font="vector" ratio="15">PE</text>
 <text x="59" y="16" size="1.778" layer="21" font="vector" ratio="15">N</text>
-<text x="233.68" y="137.16" size="3.81" layer="21" font="vector" ratio="15">&gt;PROJEKTNAME</text>
-<text x="274.32" y="137.16" size="1.778" layer="21" font="vector">v</text>
-<text x="233.68" y="134.62" size="1.778" layer="21" font="vector">&gt;AUTHOR</text>
-<text x="276.86" y="137.16" size="1.778" layer="21" font="vector">&gt;VERSION</text>
+<text x="15.5" y="40.5" size="1.778" layer="21" font="vector" ratio="15" rot="R180">PE</text>
+<text x="15.5" y="45.5" size="1.778" layer="21" font="vector" ratio="15" rot="R180">N</text>
+<text x="15.5" y="50.5" size="1.778" layer="21" font="vector" ratio="15" rot="R180">NO</text>
+<text x="15.5" y="55.5" size="1.778" layer="21" font="vector" ratio="15" rot="R180">COM</text>
+<text x="15.5" y="60.5" size="1.778" layer="21" font="vector" ratio="15" rot="R180">NC</text>
+<text x="275" y="58.5" size="1.778" layer="21" font="vector" ratio="15">NC</text>
+<text x="275" y="53.5" size="1.778" layer="21" font="vector" ratio="15">COM</text>
+<text x="275" y="48.5" size="1.778" layer="21" font="vector" ratio="15">NO</text>
+<text x="275" y="43.5" size="1.778" layer="21" font="vector" ratio="15">N</text>
+<text x="275" y="38.5" size="1.778" layer="21" font="vector" ratio="15">PE</text>
+<wire x1="0" y1="0" x2="0" y2="37" width="0" layer="20"/>
+<wire x1="0" y1="37" x2="4.5" y2="37" width="0" layer="20"/>
+<wire x1="4.5" y1="37" x2="4.5" y2="58" width="0" layer="20"/>
+<wire x1="4.5" y1="58" x2="0" y2="58" width="0" layer="20"/>
+<wire x1="0" y1="58" x2="0" y2="145" width="0" layer="20"/>
+<wire x1="290" y1="0" x2="290" y2="37" width="0" layer="20"/>
+<wire x1="290" y1="37" x2="285.5" y2="37" width="0" layer="20"/>
+<wire x1="285.5" y1="37" x2="285.5" y2="58" width="0" layer="20"/>
+<wire x1="285.5" y1="58" x2="290" y2="58" width="0" layer="20"/>
+<wire x1="290" y1="58" x2="290" y2="145" width="0" layer="20"/>
 </plain>
 <attributes>
@@
 <attribute name="MPN" value="BC846BWT1G" x="271" y="105" size="1.778" layer="27" rot="R180" display="off"/>
 </element>
+<element name="U$1" library="xMZ-Mod-Touch-Bodenplatine" package="TEXT_FUSE" value="" x="84.5" y="15"/>
+<element name="U$2" library="xMZ-Mod-Touch-Bodenplatine" package="TEXT_NAME_VERSION_AUTHOR" value="" x="236.39" y="125.88"/>
+<element name="U$3" library="xMZ-Mod-Touch-Bodenplatine" package="LOGO_RA-GAS" value="" x="227.33" y="134.62"/>
+<element name="U$4" library="xMZ-Mod-Touch-Bodenplatine" package="LOGO_RA-GAS_BOTTOM" value="" x="187.96" y="2.54"/>
+<element name="U$5" library="xMZ-Mod-Touch-Bodenplatine" package="LOGO_RA-GAS_BOTTOM" value="" x="227.33" y="2.54" rot="MR0"/>
 </elements>
 <signals>
