File: Bodenplatine v090.brd (EAGLE design)
At the start: 290 x 145 mm, 118 parts, among them K1 RY612012, K2 RY612012, K3 RY612012, K4 RY612012, K5 RY612012, K6 RY612012, K7 RY612012, K8 RY612012, K9 RY612012, Q1 BC846BLT1SMD, Q2 BC846BLT1SMD, Q3 BC846BLT1SMD, Q4 BC846BLT1SMD, Q5 BC846BLT1SMD, Q6 BC846BLT1SMD, Q7 BC846BLT1SMD, Q8 BC846BLT1SMD, Q9 BC846BLT1SMD, X1 SPRINGCON_AST125_5X2, X10 SPRINGCON_AST125_3X2, X11 SPRINGCON_AST125_4X2, X12 SPRINGCON_AST125_4X2, X13 SPRINGCON_AST125_5X2, X14 236-403, X15 236-402, X2 SPRINGCON_AST125_5X2, X3 SPRINGCON_AST125_5X2, X4 SPRINGCON_AST125_5X2, X5 SPRINGCON_AST125_5X2, X6 SPRINGCON_AST125_5X2, X7 SPRINGCON_AST125_5X2, X8 SPRINGCON_AST125_5X2, X9 SPRINGCON_AST125_5X2

Commit message: Neu versioniert, Finale Bodenplatte BETA Version
Changed lines of the file:
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@@
 <setting verticaltext="up"/>
 </settings>
-<grid distance="0.05" unitdist="inch" unit="inch" style="lines" multiple="1" display="yes" altdistance="0.005" altunitdist="inch" altunit="inch"/>
+<grid distance="0.5" unitdist="mm" unit="mm" style="lines" multiple="1" display="yes" altdistance="0.1" altunitdist="mm" altunit="mm"/>
 <layers>
 <layer number="1" name="Top" color="4" fill="1" visible="yes" active="yes"/>
@@
 <layer number="47" name="Measures" color="7" fill="1" visible="no" active="yes"/>
 <layer number="48" name="Document" color="7" fill="1" visible="no" active="yes"/>
-<layer number="49" name="Reference" color="7" fill="1" visible="yes" active="yes"/>
+<layer number="49" name="Reference" color="7" fill="1" visible="no" active="yes"/>
 <layer number="50" name="dxf" color="7" fill="1" visible="no" active="no"/>
 <layer number="51" name="tDocu" color="6" fill="1" visible="yes" active="yes"/>
@@
 <wire x1="285.5" y1="58" x2="290" y2="58" width="0" layer="20"/>
 <wire x1="290" y1="58" x2="290" y2="145" width="0" layer="20"/>
+<text x="49" y="120" size="1.778" layer="21" font="vector" ratio="15" rot="R270">+12V</text>
+<text x="53.5" y="120" size="1.778" layer="21" font="vector" ratio="15" rot="R270">GND</text>
+<wire x1="53" y1="121" x2="53" y2="112.5" width="0.254" layer="21"/>
+<wire x1="57" y1="121" x2="57.5" y2="121" width="0.254" layer="21"/>
+<wire x1="57.5" y1="121" x2="57.5" y2="112.5" width="0.254" layer="21"/>
+<wire x1="57.5" y1="112.5" x2="53" y2="112.5" width="0.254" layer="21"/>
+<wire x1="53" y1="112.5" x2="48.5" y2="112.5" width="0.254" layer="21"/>
+<wire x1="48.5" y1="112.5" x2="48.5" y2="121" width="0.254" layer="21"/>
+<text x="6.5" y="119.5" size="1.778" layer="21" font="vector" ratio="15">L</text>
+<text x="15.5" y="119.5" size="1.778" layer="21" font="vector" ratio="15">PE</text>
+<text x="11" y="119.5" size="1.778" layer="21" font="vector" ratio="15">N</text>
 </plain>
 <attributes>
