File: Deckelplatine v092.brd (EAGLE design)
At the start: 110 x 75 mm, 67 parts, among them IC1 MAX1487EESA+, IC2 74HCT595D, IC3 74HCT595D, IC4 74HCT595D, IC5 74HCT595D, IC6 74HCT595D, J1 52808-2570, Q1 BC846BSMD, Q2 BC846BSMD, U1 LM2676S, X1 236-406/000-023, X2 233-502

Commit message: Neu versioniert, Finale Bodenplatte BETA Version
Parts:
- added U$2: (no value), xMZ-Mod-Touch-Bodenplatine:LOGO_RA-GAS
- added U$3: (no value), xMZ-Mod-Touch-Bodenplatine:TEXT_NAME_VERSION_AUTHOR
Other:
- board text removed: ">VERSION"
- board text removed: "Deckelplatine"
- board text removed: "v"
Changed lines of the file:
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@@
 <layer number="54" name="bGND_GNDA" color="1" fill="9" visible="no" active="no"/>
 <layer number="56" name="wert" color="7" fill="1" visible="no" active="no"/>
+<layer number="57" name="tCAD" color="7" fill="1" visible="no" active="no"/>
+<layer number="59" name="tCarbon" color="7" fill="1" visible="no" active="no"/>
+<layer number="60" name="bCarbon" color="7" fill="1" visible="no" active="no"/>
 <layer number="90" name="Modules" color="5" fill="1" visible="no" active="no"/>
 <layer number="91" name="Nets" color="2" fill="1" visible="no" active="no"/>
@@
 <layer number="106" name="bPlate" color="7" fill="1" visible="no" active="yes"/>
 <layer number="107" name="Crop" color="7" fill="1" visible="no" active="yes"/>
+<layer number="108" name="tplace-old" color="10" fill="1" visible="no" active="yes"/>
+<layer number="109" name="ref-old" color="11" fill="1" visible="no" active="yes"/>
+<layer number="110" name="fp0" color="7" fill="1" visible="no" active="yes"/>
+<layer number="111" name="LPC17xx" color="7" fill="1" visible="no" active="yes"/>
 <layer number="112" name="bOutline" color="15" fill="11" visible="no" active="no"/>
+<layer number="113" name="IDFDebug" color="7" fill="1" visible="no" active="yes"/>
 <layer number="116" name="Patch_BOT" color="9" fill="4" visible="no" active="yes"/>
+<layer number="118" name="Rect_Pads" color="7" fill="1" visible="no" active="yes"/>
 <layer number="121" name="_tsilk" color="7" fill="1" visible="no" active="yes"/>
 <layer number="122" name="_bsilk" color="7" fill="1" visible="no" active="yes"/>
+<layer number="123" name="tTestmark" color="7" fill="1" visible="no" active="yes"/>
+<layer number="124" name="bTestmark" color="7" fill="1" visible="no" active="yes"/>
 <layer number="125" name="_tNames" color="7" fill="1" visible="no" active="yes"/>
+<layer number="126" name="_bNames" color="7" fill="1" visible="no" active="yes"/>
+<layer number="127" name="_tValues" color="7" fill="1" visible="no" active="yes"/>
+<layer number="128" name="_bValues" color="7" fill="1" visible="no" active="yes"/>
+<layer number="129" name="Mask" color="7" fill="1" visible="no" active="yes"/>
+<layer number="131" name="tAdjust" color="7" fill="1" visible="no" active="yes"/>
+<layer number="132" name="bAdjust" color="7" fill="1" visible="no" active="yes"/>
 <layer number="144" name="Drill_legend" color="7" fill="1" visible="no" active="yes"/>
 <layer number="150" name="misc1" color="7" fill="1" visible="no" active="yes"/>
 <layer number="151" name="HeatSink" color="7" fill="1" visible="no" active="yes"/>
+<layer number="152" name="_bDocu" color="7" fill="1" visible="no" active="yes"/>
+<layer number="153" name="FabDoc1" color="7" fill="1" visible="no" active="yes"/>
+<layer number="154" name="FabDoc2" color="7" fill="1" visible="no" active="yes"/>
+<layer number="155" name="FabDoc3" color="7" fill="1" visible="no" active="yes"/>
 <layer number="199" name="Contour" color="7" fill="1" visible="no" active="yes"/>
 <layer number="200" name="200bmp" color="1" fill="10" visible="no" active="yes"/>
@@
 <layer number="232" name="Eagle3D_PG2" color="7" fill="1" visible="no" active="yes"/>
 <layer number="233" name="Eagle3D_PG3" color="7" fill="1" visible="no" active="yes"/>
+<layer number="248" name="Housing" color="7" fill="1" visible="no" active="yes"/>
+<layer number="249" name="Edge" color="7" fill="1" visible="no" active="yes"/>
 <layer number="250" name="Descript" color="3" fill="1" visible="no" active="no"/>
 <layer number="251" name="SMDround" color="12" fill="11" visible="no" active="no"/>
 <layer number="254" name="cooling" color="7" fill="1" visible="no" active="yes"/>
+<layer number="255" name="routoute" color="7" fill="1" visible="no" active="yes"/>
 </layers>
 <board>
@@
 <text x="30" y="8" size="0.8" layer="21" font="vector" ratio="10">BUS Terminator</text>
 <text x="9.5932" y="72.191" size="2" layer="21" font="vector" ratio="15">xMZ-Mod-Touch</text>
-<text x="24" y="3.5" size="3.81" layer="21" font="vector" ratio="14">Deckelplatine</text>
 <text x="70.7564" y="54.4172" size="0.8" layer="21" font="vector" ratio="5">Monitor-Batterie</text>
 <text x="84.1722" y="54.341" size="0.8" layer="21" font="vector" ratio="5">Monitor-Mains</text>
@@
 <text x="91.29" y="71.45" size="1.778" layer="22" font="vector" ratio="15">+</text>
 <text x="87.374" y="71.485" size="1.778" layer="22" font="vector" ratio="15">-</text>
-<text x="67.5" y="3.5" size="1.778" layer="21" font="vector" ratio="15">&gt;VERSION</text>
-<text x="65.5" y="3.5" size="1.778" layer="21" font="vector" ratio="15">v</text>
 <text x="33.0442" y="62.4878" size="1.778" layer="21" font="vector" ratio="15">630mA</text>
 <circle x="68.9864" y="56.0832" radius="1.27" width="0.3048" layer="21"/>
@@
 </plain>
 <attributes>
-<attribute name="VERSION" value="0.9.1"/>
+<attribute name="AUTHOR" value="Stefan Müller"/>
+<attribute name="PROJEKTNAME" value="Deckelplatine"/>
+<attribute name="VERSION" value="0.9.2"/>
 </attributes>
 <variantdefs>
@@
 <attribute name="MPN" value="" x="69" y="56" size="1.778" layer="27" display="off"/>
 </element>
+<element name="U$2" library="xMZ-Mod-Touch-Bodenplatine" package="LOGO_RA-GAS" value="" x="62.23" y="0"/>
+<element name="U$3" library="xMZ-Mod-Touch-Bodenplatine" package="TEXT_NAME_VERSION_AUTHOR" value="" x="8.89" y="0"/>
 </elements>
 <signals>
