File: Bodenplatine.brd (EAGLE design)
At the start: 290 x 145 mm, 118 parts, among them K1 RY612012, K2 RY612012, K3 RY612012, K4 RY612012, K5 RY612012, K6 RY612012, K7 RY612012, K8 RY612012, K9 RY612012, Q1 BC846BLT1SMD, Q2 BC846BLT1SMD, Q3 BC846BLT1SMD, Q4 BC846BLT1SMD, Q5 BC846BLT1SMD, Q6 BC846BLT1SMD, Q7 BC846BLT1SMD, Q8 BC846BLT1SMD, Q9 BC846BLT1SMD, X1 SPRINGCON_AST125_5X2, X10 SPRINGCON_AST125_3X2, X11 SPRINGCON_AST125_4X2, X12 SPRINGCON_AST125_4X2, X13 SPRINGCON_AST125_5X2, X14 236-403, X15 236-402, X2 SPRINGCON_AST125_5X2, X3 SPRINGCON_AST125_5X2, X4 SPRINGCON_AST125_5X2, X5 SPRINGCON_AST125_5X2, X6 SPRINGCON_AST125_5X2, X7 SPRINGCON_AST125_5X2, X8 SPRINGCON_AST125_5X2, X9 SPRINGCON_AST125_5X2

Commit message: Fix 12V Spannungsversorgung vergessen ><
Connections:
- removed net N$11: K2.A1, V6.C
- removed net N$17: K3.A1, V7.C
- removed net N$27: K4.A1, V8.C
- removed net N$37: K5.A1, V13.C
- removed net N$47: K6.A1, V14.C
- removed net N$57: K7.A1, V15.C
- removed net N$67: K8.A1, V16.C
- removed net N$77: K9.A1, V18.C
- removed net N$87: K1.A1, V5.C
- net 12V: now also K1.A1, K2.A1, K3.A1, K4.A1, K5.A1, K6.A1, K7.A1, K8.A1, K9.A1, V13.C, V14.C, V15.C, V16.C, V18.C, V5.C, V6.C, V7.C, V8.C
Routing:
- net 12V: track 498.9 -> 875.3 mm
- net N$77: track 5.17 -> 0.00 mm
- net N$67: track 5.17 -> 0.00 mm
- net N$57: track 5.17 -> 0.00 mm
- net N$47: track 5.17 -> 0.00 mm
- net N$37: track 5.17 -> 0.00 mm
- net N$27: track 5.17 -> 0.00 mm
- net N$17: track 5.17 -> 0.00 mm
- net N$11: track 5.17 -> 0.00 mm
- net N$87: track 5.17 -> 0.00 mm
Changed lines of the file:
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@@
 <setting verticaltext="up"/>
 </settings>
-<grid distance="0.5" unitdist="mm" unit="mm" style="lines" multiple="1" display="yes" altdistance="0.1" altunitdist="mm" altunit="mm"/>
+<grid distance="0.05" unitdist="inch" unit="inch" style="lines" multiple="1" display="yes" altdistance="0.005" altunitdist="inch" altunit="inch"/>
 <layers>
 <layer number="1" name="Top" color="4" fill="1" visible="yes" active="yes"/>
@@
 <layer number="23" name="tOrigins" color="15" fill="1" visible="yes" active="yes"/>
 <layer number="24" name="bOrigins" color="15" fill="1" visible="yes" active="yes"/>
-<layer number="25" name="tNames" color="7" fill="1" visible="yes" active="yes"/>
+<layer number="25" name="tNames" color="7" fill="1" visible="no" active="yes"/>
 <layer number="26" name="bNames" color="7" fill="1" visible="no" active="yes"/>
 <layer number="27" name="tValues" color="7" fill="1" visible="no" active="yes"/>
@@
 <attribute name="AUTHOR" value="Stefan Müller"/>
 <attribute name="PROJEKTNAME" value="Bodenplatine"/>
-<attribute name="VERSION" value="0.0.1"/>
+<attribute name="VERSION" value="0.9.2"/>
 </attributes>
 <variantdefs>
@@
 <wire x1="61.5" y1="60.5" x2="61" y2="60" width="2.54" layer="16"/>
 </signal>
-<signal name="N$11">
-<contactref element="V6" pad="C"/>
-<contactref element="K2" pad="A1"/>
-<wire x1="59.94" y1="97.7" x2="59.94" y2="99.89" width="0.6096" layer="1"/>
-<wire x1="59.94" y1="99.89" x2="62.05" y2="102" width="0.6096" layer="1"/>
-</signal>
 <signal name="PE">
 <contactref element="X2" pad="5"/>
@@
 <wire x1="99.45" y1="109.9" x2="99.35" y2="110" width="0.6096" layer="1"/>
 </signal>
-<signal name="N$17">
-<contactref element="V7" pad="C"/>
-<contactref element="K3" pad="A1"/>
-<wire x1="88.69" y1="97.7" x2="88.69" y2="99.89" width="0.6096" layer="1"/>
-<wire x1="88.69" y1="99.89" x2="90.8" y2="102" width="0.6096" layer="1"/>
-</signal>
 <signal name="N$18">
 <contactref element="V7" pad="A"/>
@@
 <wire x1="128.2" y1="109.9" x2="128.1" y2="110" width="0.6096" layer="1"/>
 </signal>
-<signal name="N$27">
-<contactref element="V8" pad="C"/>
-<contactref element="K4" pad="A1"/>
-<wire x1="117.44" y1="97.7" x2="117.44" y2="99.89" width="0.6096" layer="1"/>
-<wire x1="117.44" y1="99.89" x2="119.55" y2="102" width="0.6096" layer="1"/>
-</signal>
 <signal name="N$28">
 <contactref element="V8" pad="A"/>
@@
 <wire x1="156.95" y1="109.9" x2="156.85" y2="110" width="0.6096" layer="1"/>
 </signal>
-<signal name="N$37">
-<contactref element="V13" pad="C"/>
-<contactref element="K5" pad="A1"/>
-<wire x1="146.19" y1="97.7" x2="146.19" y2="99.89" width="0.6096" layer="1"/>
-<wire x1="146.19" y1="99.89" x2="148.3" y2="102" width="0.6096" layer="1"/>
-</signal>
 <signal name="N$38">
 <contactref element="V13" pad="A"/>
@@
 <wire x1="185.7" y1="106.1" x2="185.7" y2="109.9" width="0.6096" layer="1"/>
 <wire x1="185.7" y1="109.9" x2="185.6" y2="110" width="0.6096" layer="1"/>
-</signal>
-<signal name="N$47">
-<contactref element="V14" pad="C"/>
-<contactref element="K6" pad="A1"/>
-<wire x1="174.94" y1="97.7" x2="174.94" y2="99.89" width="0.6096" layer="1"/>
-<wire x1="174.94" y1="99.89" x2="177.05" y2="102" width="0.6096" layer="1"/>
 </signal>
 <signal name="N$48">
@@
 <wire x1="214.45" y1="109.9" x2="214.35" y2="110" width="0.6096" layer="1"/>
 </signal>
-<signal name="N$57">
-<contactref element="V15" pad="C"/>
-<contactref element="K7" pad="A1"/>
-<wire x1="203.69" y1="97.7" x2="203.69" y2="99.89" width="0.6096" layer="1"/>
-<wire x1="203.69" y1="99.89" x2="205.8" y2="102" width="0.6096" layer="1"/>
-</signal>
 <signal name="N$58">
 <contactref element="V15" pad="A"/>
@@
 <wire x1="243.2" y1="109.9" x2="243.1" y2="110" width="0.6096" layer="1"/>
 </signal>
-<signal name="N$67">
-<contactref element="V16" pad="C"/>
-<contactref element="K8" pad="A1"/>
-<wire x1="232.44" y1="97.7" x2="232.44" y2="99.89" width="0.6096" layer="1"/>
-<wire x1="232.44" y1="99.89" x2="234.55" y2="102" width="0.6096" layer="1"/>
-</signal>
 <signal name="N$68">
 <contactref element="V16" pad="A"/>
@@
 <wire x1="271.95" y1="106.1" x2="271.95" y2="109.9" width="0.6096" layer="1"/>
 <wire x1="271.95" y1="109.9" x2="271.85" y2="110" width="0.6096" layer="1"/>
-</signal>
-<signal name="N$77">
-<contactref element="V18" pad="C"/>
-<contactref element="K9" pad="A1"/>
-<wire x1="261.19" y1="97.7" x2="261.19" y2="99.89" width="0.6096" layer="1"/>
-<wire x1="261.19" y1="99.89" x2="263.3" y2="102" width="0.6096" layer="1"/>
 </signal>
 <signal name="N$78">
@@
 <wire x1="41.95" y1="106.1" x2="41.95" y2="109.9" width="0.6096" layer="1"/>
 <wire x1="41.95" y1="109.9" x2="41.85" y2="110" width="0.6096" layer="1"/>
-</signal>
-<signal name="N$87">
-<contactref element="V5" pad="C"/>
-<contactref element="K1" pad="A1"/>
-<wire x1="31.19" y1="97.7" x2="31.19" y2="99.89" width="0.6096" layer="1"/>
-<wire x1="31.19" y1="99.89" x2="33.3" y2="102" width="0.6096" layer="1"/>
 </signal>
 <signal name="N$88">
@@
 <wire x1="281.94" y1="88.9" x2="281.94" y2="38.1" width="2.54" layer="16"/>
 <wire x1="281.94" y1="38.1" x2="275.59" y2="31.75" width="2.54" layer="16"/>
+<contactref element="V18" pad="C"/>
+<contactref element="K9" pad="A1"/>
+<wire x1="261.19" y1="97.7" x2="261.19" y2="99.89" width="0.6096" layer="1"/>
+<wire x1="261.19" y1="99.89" x2="263.3" y2="102" width="0.6096" layer="1"/>
+<contactref element="V13" pad="C"/>
+<contactref element="K5" pad="A1"/>
+<wire x1="146.19" y1="97.7" x2="146.19" y2="99.89" width="0.6096" layer="1"/>
+<wire x1="146.19" y1="99.89" x2="148.3" y2="102" width="0.6096" layer="1"/>
+<contactref element="V14" pad="C"/>
+<contactref element="K6" pad="A1"/>
+<wire x1="174.94" y1="97.7" x2="174.94" y2="99.89" width="0.6096" layer="1"/>
+<wire x1="174.94" y1="99.89" x2="177.05" y2="102" width="0.6096" layer="1"/>
+<contactref element="V15" pad="C"/>
+<contactref element="K7" pad="A1"/>
+<wire x1="203.69" y1="97.7" x2="203.69" y2="99.89" width="0.6096" layer="1"/>
+<wire x1="203.69" y1="99.89" x2="205.8" y2="102" width="0.6096" layer="1"/>
+<contactref element="V16" pad="C"/>
+<contactref element="K8" pad="A1"/>
+<wire x1="232.44" y1="97.7" x2="232.44" y2="99.89" width="0.6096" layer="1"/>
+<wire x1="232.44" y1="99.89" x2="234.55" y2="102" width="0.6096" layer="1"/>
+<contactref element="V8" pad="C"/>
+<contactref element="K4" pad="A1"/>
+<wire x1="117.44" y1="97.7" x2="117.44" y2="99.89" width="0.6096" layer="1"/>
+<wire x1="117.44" y1="99.89" x2="119.55" y2="102" width="0.6096" layer="1"/>
+<contactref element="V7" pad="C"/>
+<contactref element="K3" pad="A1"/>
+<wire x1="88.69" y1="97.7" x2="88.69" y2="99.89" width="0.6096" layer="1"/>
+<wire x1="88.69" y1="99.89" x2="90.8" y2="102" width="0.6096" layer="1"/>
+<contactref element="V6" pad="C"/>
+<contactref element="K2" pad="A1"/>
+<wire x1="59.94" y1="97.7" x2="59.94" y2="99.89" width="0.6096" layer="1"/>
+<wire x1="59.94" y1="99.89" x2="62.05" y2="102" width="0.6096" layer="1"/>
+<contactref element="V5" pad="C"/>
+<contactref element="K1" pad="A1"/>
+<wire x1="31.19" y1="97.7" x2="31.19" y2="99.89" width="0.6096" layer="1"/>
+<wire x1="31.19" y1="99.89" x2="33.3" y2="102" width="0.6096" layer="1"/>
+<wire x1="261.19" y1="97.7" x2="261.19" y2="94.82" width="2.54" layer="1"/>
+<wire x1="261.19" y1="94.82" x2="259.08" y2="92.71" width="2.54" layer="1"/>
+<wire x1="259.08" y1="92.71" x2="233.68" y2="92.71" width="2.54" layer="1"/>
+<wire x1="233.68" y1="92.71" x2="204.47" y2="92.71" width="2.54" layer="1"/>
+<wire x1="204.47" y1="92.71" x2="176.53" y2="92.71" width="2.54" layer="1"/>
+<wire x1="176.53" y1="92.71" x2="147.32" y2="92.71" width="2.54" layer="1"/>
+<wire x1="147.32" y1="92.71" x2="119.38" y2="92.71" width="2.54" layer="1"/>
+<wire x1="119.38" y1="92.71" x2="91.44" y2="92.71" width="2.54" layer="1"/>
+<wire x1="91.44" y1="92.71" x2="62.23" y2="92.71" width="2.54" layer="1"/>
+<wire x1="62.23" y1="92.71" x2="33.02" y2="92.71" width="2.54" layer="1"/>
+<wire x1="59.94" y1="97.7" x2="59.94" y2="95" width="2.54" layer="1"/>
+<wire x1="59.94" y1="95" x2="62.23" y2="92.71" width="2.54" layer="1"/>
+<wire x1="88.69" y1="97.7" x2="88.69" y2="95.46" width="2.54" layer="1"/>
+<wire x1="88.69" y1="95.46" x2="91.44" y2="92.71" width="2.54" layer="1"/>
+<wire x1="117.44" y1="97.7" x2="117.44" y2="94.65" width="2.54" layer="1"/>
+<wire x1="117.44" y1="94.65" x2="119.38" y2="92.71" width="0.6096" layer="1"/>
+<wire x1="146.19" y1="97.7" x2="146.19" y2="93.84" width="2.54" layer="1"/>
+<wire x1="146.19" y1="93.84" x2="147.32" y2="92.71" width="0.6096" layer="1"/>
+<wire x1="174.94" y1="97.7" x2="174.94" y2="94.3" width="2.54" layer="1"/>
+<wire x1="174.94" y1="94.3" x2="176.53" y2="92.71" width="0.6096" layer="1"/>
+<wire x1="232.44" y1="97.7" x2="232.44" y2="93.95" width="2.54" layer="1"/>
+<wire x1="232.44" y1="93.95" x2="233.68" y2="92.71" width="0.6096" layer="1"/>
+<wire x1="203.69" y1="97.7" x2="203.69" y2="93.49" width="2.54" layer="1"/>
+<wire x1="203.69" y1="93.49" x2="204.47" y2="92.71" width="0.6096" layer="1"/>
+<wire x1="31.19" y1="97.7" x2="28.03" y2="97.7" width="2.54" layer="1"/>
+<wire x1="28.03" y1="97.7" x2="26.67" y2="99.06" width="2.54" layer="1"/>
+<wire x1="26.67" y1="99.06" x2="26.67" y2="119.38" width="2.54" layer="1"/>
+<wire x1="26.67" y1="119.38" x2="31.75" y2="124.46" width="2.54" layer="1"/>
+<wire x1="31.75" y1="124.46" x2="49.53" y2="124.46" width="2.54" layer="1"/>
+<wire x1="50.65" y1="125.9573" x2="50.65" y2="125.58" width="0.6096" layer="1"/>
+<wire x1="50.65" y1="125.58" x2="49.53" y2="124.46" width="2.54" layer="1"/>
+<wire x1="31.19" y1="97.7" x2="31.19" y2="94.54" width="2.54" layer="1"/>
+<wire x1="31.19" y1="94.54" x2="33.02" y2="92.71" width="2.54" layer="1"/>
 </signal>
 <signal name="A-">
