File: Bodenplatine.brd (EAGLE design)
At the start: 290 x 145 mm, 118 parts, among them K1 RY612012, K2 RY612012, K3 RY612012, K4 RY612012, K5 RY612012, K6 RY612012, K7 RY612012, K8 RY612012, K9 RY612012, Q1 BC846BLT1SMD, Q2 BC846BLT1SMD, Q3 BC846BLT1SMD, Q4 BC846BLT1SMD, Q5 BC846BLT1SMD, Q6 BC846BLT1SMD, Q7 BC846BLT1SMD, Q8 BC846BLT1SMD, Q9 BC846BLT1SMD, X1 SPRINGCON_AST125_5X2, X10 SPRINGCON_AST125_3X2, X11 SPRINGCON_AST125_4X2, X12 SPRINGCON_AST125_4X2, X13 SPRINGCON_AST125_5X2, X14 236-403, X15 236-402, X2 SPRINGCON_AST125_5X2, X3 SPRINGCON_AST125_5X2, X4 SPRINGCON_AST125_5X2, X5 SPRINGCON_AST125_5X2, X6 SPRINGCON_AST125_5X2, X7 SPRINGCON_AST125_5X2, X8 SPRINGCON_AST125_5X2, X9 SPRINGCON_AST125_5X2

Commit message: Kosmetische Verbesserungen
Parts:
- H1, H2, H3, H4: value MOUNT-HOLE3.3 -> MOUNT-PAD-ROUND3.3; device holes:3,3 -> holes:3,3-PAD
- moved U$2 44.4 mm to (191.9, 125.9)
- moved U$3 35.6 mm to (191.8, 134.6)
Connections:
- net GND: now also H1.B3,3, H2.B3,3, H3.B3,3, H4.B3,3
Routing:
- net B+: track 269.2 -> 270.2 mm
- net A-: track 271.9 -> 272.9 mm
- net 12V: track 875.3 -> 875.8 mm
