File: Bodenplatine.brd (EAGLE design)
At the start: 290 x 145 mm, 118 parts, among them K1 RY612012, K2 RY612012, K3 RY612012, K4 RY612012, K5 RY612012, K6 RY612012, K7 RY612012, K8 RY612012, K9 RY612012, Q1 BC846BLT1SMD, Q2 BC846BLT1SMD, Q3 BC846BLT1SMD, Q4 BC846BLT1SMD, Q5 BC846BLT1SMD, Q6 BC846BLT1SMD, Q7 BC846BLT1SMD, Q8 BC846BLT1SMD, Q9 BC846BLT1SMD, X1 SPRINGCON_AST125_5X2, X10 SPRINGCON_AST125_3X2, X11 SPRINGCON_AST125_4X2, X12 SPRINGCON_AST125_4X2, X13 SPRINGCON_AST125_5X2, X14 236-403, X15 236-402, X2 SPRINGCON_AST125_5X2, X3 SPRINGCON_AST125_5X2, X4 SPRINGCON_AST125_5X2, X5 SPRINGCON_AST125_5X2, X6 SPRINGCON_AST125_5X2, X7 SPRINGCON_AST125_5X2, X8 SPRINGCON_AST125_5X2, X9 SPRINGCON_AST125_5X2

Commit message: A3 Rahmen in BRD eingefügt
Parts:
- U$4: device xMZ-Mod-Touch-Bodenplatine:LOGO_RA-GAS_BOTTOM -> xMZ-Mod-Touch-Bodenplatine:LOGO_RA-GAS_TOP
- U$5: device xMZ-Mod-Touch-Bodenplatine:LOGO_RA-GAS_BOTTOM -> xMZ-Mod-Touch-Bodenplatine:A3-LOC-RA-GAS
- moved U$5 112.1 mm to (135.9, 67.3), flipped to the top
- moved U$4 2.96 mm to (188.0, 5.50)
Other:
- outline, holes or cut-outs redrawn
- board text added: "12V"
- board text added: "5V"
- board text added: "P1"
- board text added: "P2"
- board text added: "P3"
- board text added: "P4"
- board text added: "P5"
- board text added: "P6"
- board text added: "P7"
- board text added: "P8"
- board text added: "P9"
Changed lines of the file:
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@@
 <setting verticaltext="up"/>
 </settings>
-<grid distance="0.05" unitdist="inch" unit="mic" style="lines" multiple="1" display="yes" altdistance="0.005" altunitdist="inch" altunit="inch"/>
+<grid distance="0.05" unitdist="inch" unit="inch" style="lines" multiple="1" display="yes" altdistance="0.005" altunitdist="inch" altunit="inch"/>
 <layers>
-<layer number="1" name="Top" color="4" fill="1" visible="yes" active="yes"/>
+<layer number="1" name="Top" color="4" fill="1" visible="no" active="yes"/>
 <layer number="2" name="Route2" color="1" fill="3" visible="no" active="no"/>
 <layer number="3" name="Route3" color="4" fill="3" visible="no" active="no"/>
@@
 <layer number="14" name="Route14" color="1" fill="6" visible="no" active="no"/>
 <layer number="15" name="Route15" color="4" fill="6" visible="no" active="no"/>
-<layer number="16" name="Bottom" color="1" fill="1" visible="yes" active="yes"/>
+<layer number="16" name="Bottom" color="1" fill="1" visible="no" active="yes"/>
 <layer number="17" name="Pads" color="2" fill="1" visible="yes" active="yes"/>
-<layer number="18" name="Vias" color="2" fill="1" visible="yes" active="yes"/>
-<layer number="19" name="Unrouted" color="6" fill="1" visible="yes" active="yes"/>
+<layer number="18" name="Vias" color="2" fill="1" visible="no" active="yes"/>
+<layer number="19" name="Unrouted" color="6" fill="1" visible="no" active="yes"/>
 <layer number="20" name="Dimension" color="15" fill="1" visible="yes" active="yes"/>
 <layer number="21" name="tPlace" color="16" fill="1" visible="yes" active="yes"/>
-<layer number="22" name="bPlace" color="14" fill="1" visible="yes" active="yes"/>
+<layer number="22" name="bPlace" color="14" fill="1" visible="no" active="yes"/>
 <layer number="23" name="tOrigins" color="15" fill="1" visible="yes" active="yes"/>
-<layer number="24" name="bOrigins" color="15" fill="1" visible="yes" active="yes"/>
-<layer number="25" name="tNames" color="7" fill="1" visible="no" active="yes"/>
+<layer number="24" name="bOrigins" color="15" fill="1" visible="no" active="yes"/>
+<layer number="25" name="tNames" color="7" fill="1" visible="yes" active="yes"/>
 <layer number="26" name="bNames" color="7" fill="1" visible="no" active="yes"/>
 <layer number="27" name="tValues" color="7" fill="1" visible="no" active="yes"/>
@@
 <layer number="29" name="tStop" color="7" fill="3" visible="no" active="yes"/>
 <layer number="30" name="bStop" color="7" fill="6" visible="no" active="yes"/>
-<layer number="31" name="tCream" color="7" fill="4" visible="no" active="yes"/>
+<layer number="31" name="tCream" color="7" fill="4" visible="yes" active="yes"/>
 <layer number="32" name="bCream" color="7" fill="5" visible="no" active="yes"/>
 <layer number="33" name="tFinish" color="6" fill="3" visible="no" active="yes"/>
@@
 <layer number="42" name="bRestrict" color="1" fill="10" visible="no" active="yes"/>
 <layer number="43" name="vRestrict" color="2" fill="10" visible="no" active="yes"/>
-<layer number="44" name="Drills" color="7" fill="1" visible="no" active="yes"/>
+<layer number="44" name="Drills" color="7" fill="1" visible="yes" active="yes"/>
 <layer number="45" name="Holes" color="7" fill="1" visible="yes" active="yes"/>
 <layer number="46" name="Milling" color="3" fill="1" visible="no" active="yes"/>
-<layer number="47" name="Measures" color="7" fill="1" visible="no" active="yes"/>
-<layer number="48" name="Document" color="7" fill="1" visible="no" active="yes"/>
+<layer number="47" name="Measures" color="7" fill="1" visible="yes" active="yes"/>
+<layer number="48" name="Document" color="7" fill="1" visible="yes" active="yes"/>
 <layer number="49" name="Reference" color="7" fill="1" visible="no" active="yes"/>
 <layer number="50" name="dxf" color="7" fill="1" visible="no" active="no"/>
@@
 <layer number="154" name="FabDoc2" color="7" fill="1" visible="no" active="yes"/>
 <layer number="155" name="FabDoc3" color="7" fill="1" visible="no" active="yes"/>
-<layer number="160" name="BlindViaText" color="6" fill="1" visible="yes" active="yes"/>
-<layer number="161" name="BlindViaDraw" color="6" fill="1" visible="yes" active="yes"/>
+<layer number="160" name="BlindViaText" color="6" fill="1" visible="no" active="yes"/>
+<layer number="161" name="BlindViaDraw" color="6" fill="1" visible="no" active="yes"/>
 <layer number="199" name="Contour" color="7" fill="1" visible="no" active="yes"/>
 <layer number="200" name="200bmp" color="1" fill="10" visible="no" active="yes"/>
@@
 <text x="275" y="43.5" size="1.778" layer="21" font="vector" ratio="15">N</text>
 <text x="275" y="38.5" size="1.778" layer="21" font="vector" ratio="15">PE</text>
-<wire x1="0" y1="0" x2="0" y2="37" width="0" layer="20"/>
-<wire x1="0" y1="37" x2="4.5" y2="37" width="0" layer="20"/>
-<wire x1="4.5" y1="37" x2="4.5" y2="58" width="0" layer="20"/>
+<wire x1="0" y1="0" x2="0" y2="42" width="0" layer="20"/>
+<wire x1="0" y1="42" x2="4.5" y2="42" width="0" layer="20"/>
+<wire x1="4.5" y1="42" x2="4.5" y2="58" width="0" layer="20"/>
 <wire x1="4.5" y1="58" x2="0" y2="58" width="0" layer="20"/>
 <wire x1="0" y1="58" x2="0" y2="145" width="0" layer="20"/>
-<wire x1="290" y1="0" x2="290" y2="37" width="0" layer="20"/>
-<wire x1="290" y1="37" x2="285.5" y2="37" width="0" layer="20"/>
-<wire x1="285.5" y1="37" x2="285.5" y2="58" width="0" layer="20"/>
+<wire x1="290" y1="0" x2="290" y2="42" width="0" layer="20"/>
+<wire x1="290" y1="42" x2="285.5" y2="42" width="0" layer="20"/>
+<wire x1="285.5" y1="42" x2="285.5" y2="58" width="0" layer="20"/>
 <wire x1="285.5" y1="58" x2="290" y2="58" width="0" layer="20"/>
 <wire x1="290" y1="58" x2="290" y2="145" width="0" layer="20"/>
@@
 <text x="270.20625" y="106.1390625" size="0.05" layer="160" font="vector" ratio="15" rot="R10">FillOverPAD:GND:161:420</text>
 <wire x1="270.05" y1="106.1" x2="270.20625" y2="106.1390625" width="0.025" layer="160"/>
+<text x="132.7" y="131.08" size="1.016" layer="21" font="vector" rot="R270">P4</text>
+<text x="135.24" y="131.08" size="1.016" layer="21" font="vector" rot="R270">P5</text>
+<text x="137.78" y="131.08" size="1.016" layer="21" font="vector" rot="R270">P6</text>
+<text x="140.32" y="131.08" size="1.016" layer="21" font="vector" rot="R270">GND</text>
+<text x="142.86" y="131.08" size="1.016" layer="21" font="vector" rot="R270">5V</text>
+<text x="145.4" y="131.08" size="1.016" layer="21" font="vector" rot="R270">P7</text>
+<text x="147.94" y="131.08" size="1.016" layer="21" font="vector" rot="R270">P8</text>
+<text x="150.48" y="131.08" size="1.016" layer="21" font="vector" rot="R270">P9</text>
+<text x="155.56" y="131.08" size="1.016" layer="21" font="vector" rot="R270">B+</text>
+<text x="134" y="139.43" size="1.016" layer="21" font="vector" rot="R90">P3</text>
+<text x="136.54" y="139.43" size="1.016" layer="21" font="vector" rot="R90">P2</text>
+<text x="139.08" y="139.43" size="1.016" layer="21" font="vector" rot="R90">P1</text>
+<text x="141.62" y="139.43" size="1.016" layer="21" font="vector" rot="R90">GND</text>
+<text x="144.16" y="139.43" size="1.016" layer="21" font="vector" rot="R90">5V</text>
+<text x="146.7" y="139.43" size="1.016" layer="21" font="vector" rot="R90">12V</text>
+<text x="156.86" y="139.43" size="1.016" layer="21" font="vector" rot="R90">A-</text>
 </plain>
 <attributes>
 <attribute name="AUTHOR" value="Stefan Müller"/>
+<attribute name="DESCRIPTION" value="Placement"/>
 <attribute name="PROJEKTNAME" value="xMZ-Mod-Touch-Bodenplatine"/>
 <attribute name="VERSION" value="0.9.5"/>
@@
 <attribute name="MPN" value="" x="45" y="18" size="1.778" layer="27" display="off"/>
 </element>
-<element name="JP1" library="pinhead" package="2X10" value="Stiftleiste 2x20 pol" x="145" y="135">
+<element name="JP1" library="pinhead" package="2X10" value="Stiftleiste 2x20 pol" x="145" y="135" smashed="yes">
 <attribute name="OC_FARNELL" value="3417773" x="145" y="135" size="1.778" layer="27" display="off"/>
 <attribute name="MF" value="TE CONNECTIVITY / AMP" x="145" y="135" size="1.778" layer="27" display="off"/>
 <attribute name="MPN" value="825440-5" x="145" y="135" size="1.778" layer="27" display="off"/>
+<attribute name="NAME" x="129.325" y="135.3" size="1.27" layer="25" ratio="10" rot="R90"/>
+<attribute name="VALUE" x="132.3" y="130.555" size="1.27" layer="27"/>
 </element>
 <element name="R2" library="rcl" package="M0805" value="270R" x="73.75" y="117" rot="R90">
@@
 <attribute name="MF" value="WAGO" x="53" y="128" size="1.778" layer="27" rot="R90" display="off"/>
 <attribute name="MPN" value="236-402" x="53" y="128" size="1.778" layer="27" rot="R90" display="off"/>
-<attribute name="NAME" x="46.27" y="130.4073" size="2" layer="25" font="vector" ratio="10" rot="R90"/>
+<attribute name="NAME" x="46.27" y="121.4073" size="2" layer="25" font="vector" ratio="10" rot="R90"/>
 <attribute name="VALUE" x="62.19" y="123.9173" size="2" layer="27" font="vector" ratio="10" rot="R90"/>
 </element>
@@
 <element name="U$2" library="xMZ-Mod-Touch-Bodenplatine" package="TEXT_NAME_VERSION_AUTHOR" value="" x="191.94" y="125.88"/>
 <element name="U$3" library="xMZ-Mod-Touch-Bodenplatine" package="LOGO_RA-GAS" value="" x="191.77" y="134.62"/>
-<element name="U$4" library="xMZ-Mod-Touch-Bodenplatine" package="LOGO_RA-GAS_BOTTOM" value="" x="187.96" y="2.54"/>
-<element name="U$5" library="xMZ-Mod-Touch-Bodenplatine" package="LOGO_RA-GAS_BOTTOM" value="" x="227.33" y="2.54" rot="MR0"/>
+<element name="U$4" library="xMZ-Mod-Touch-Bodenplatine" package="LOGO_RA-GAS_TOP" value="" x="188" y="5.5"/>
+<element name="U$5" library="xMZ-Mod-Touch-Bodenplatine" package="A3-LOC-RA-GAS" value="" x="135.89" y="67.31"/>
 </elements>
 <signals>
