File: Bodenplatine.sch (EAGLE design)
At the start: 113 parts, among them K1 RY612012, K2 RY612012, K3 RY612012, K4 RY612012, K5 RY612012, K6 RY612012, K7 RY612012, K8 RY612012, K9 RY612012, Q1 BC846BLT1SMD, Q2 BC846BLT1SMD, Q3 BC846BLT1SMD, Q4 BC846BLT1SMD, Q5 BC846BLT1SMD, Q6 BC846BLT1SMD, Q7 BC846BLT1SMD, Q8 BC846BLT1SMD, Q9 BC846BLT1SMD, X1 SPRINGCON_AST125_5X2, X10 SPRINGCON_AST125_3X2, X11 SPRINGCON_AST125_4X2, X12 SPRINGCON_AST125_4X2, X13 SPRINGCON_AST125_5X2, X14 236-403, X15 236-402, X2 SPRINGCON_AST125_5X2, X3 SPRINGCON_AST125_5X2, X4 SPRINGCON_AST125_5X2, X5 SPRINGCON_AST125_5X2, X6 SPRINGCON_AST125_5X2, X7 SPRINGCON_AST125_5X2, X8 SPRINGCON_AST125_5X2, X9 SPRINGCON_AST125_5X2

Commit message: Kosmetische Verbesserungen
Parts:
- H1, H2, H3, H4: value MOUNT-HOLE3.3 -> MOUNT-PAD-ROUND3.3; device holes:MOUNT-HOLE3.3 -> holes:MOUNT-PAD-ROUND3.3
Connections:
- net GND: now also H1.MOUNT, H2.MOUNT, H3.MOUNT, H4.MOUNT
Other:
- moved on the sheet: H1, H2, H3, H4
Changed lines of the file:
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@@
 <attribute name="AUTHOR" value="Stefan Müller"/>
 <attribute name="PROJEKTNAME" value="xMZ-Mod-Touch-Bodenplatine"/>
-<attribute name="VERSION" value="0.9.2"/>
+<attribute name="VERSION" value="0.9.5"/>
 </attributes>
 <variantdefs>
@@
 <attribute name="OC_FARNELL" value="1283526"/>
 </part>
-<part name="H4" library="holes" deviceset="MOUNT-HOLE" device="3.3">
-<attribute name="MF" value=""/>
-<attribute name="MPN" value=""/>
-<attribute name="OC_FARNELL" value="unknown"/>
-</part>
-<part name="H3" library="holes" deviceset="MOUNT-HOLE" device="3.3">
-<attribute name="MF" value=""/>
-<attribute name="MPN" value=""/>
-<attribute name="OC_FARNELL" value="unknown"/>
-</part>
-<part name="H2" library="holes" deviceset="MOUNT-HOLE" device="3.3">
-<attribute name="MF" value=""/>
-<attribute name="MPN" value=""/>
-<attribute name="OC_FARNELL" value="unknown"/>
-</part>
-<part name="H1" library="holes" deviceset="MOUNT-HOLE" device="3.3">
+<part name="H4" library="holes" deviceset="MOUNT-PAD-ROUND" device="3.3">
+<attribute name="MF" value=""/>
+<attribute name="MPN" value=""/>
+<attribute name="OC_FARNELL" value="unknown"/>
+</part>
+<part name="H3" library="holes" deviceset="MOUNT-PAD-ROUND" device="3.3">
+<attribute name="MF" value=""/>
+<attribute name="MPN" value=""/>
+<attribute name="OC_FARNELL" value="unknown"/>
+</part>
+<part name="H2" library="holes" deviceset="MOUNT-PAD-ROUND" device="3.3">
+<attribute name="MF" value=""/>
+<attribute name="MPN" value=""/>
+<attribute name="OC_FARNELL" value="unknown"/>
+</part>
+<part name="H1" library="holes" deviceset="MOUNT-PAD-ROUND" device="3.3">
 <attribute name="MF" value=""/>
 <attribute name="MPN" value=""/>
@@
 <attribute name="MPN" x="350.52" y="144.78" size="1.27" layer="96" display="off"/>
 </instance>
-<instance part="H4" gate="G$1" x="10.16" y="10.16">
-<attribute name="OC_FARNELL" x="10.16" y="10.16" size="1.27" layer="96" display="off"/>
-<attribute name="MF" x="10.16" y="10.16" size="1.27" layer="96" display="off"/>
-<attribute name="MPN" x="10.16" y="10.16" size="1.27" layer="96" display="off"/>
-</instance>
-<instance part="H3" gate="G$1" x="10.16" y="17.78">
-<attribute name="OC_FARNELL" x="10.16" y="17.78" size="1.27" layer="96" display="off"/>
-<attribute name="MF" x="10.16" y="17.78" size="1.27" layer="96" display="off"/>
-<attribute name="MPN" x="10.16" y="17.78" size="1.27" layer="96" display="off"/>
-</instance>
-<instance part="H2" gate="G$1" x="10.16" y="25.4">
-<attribute name="OC_FARNELL" x="10.16" y="25.4" size="1.27" layer="96" display="off"/>
-<attribute name="MF" x="10.16" y="25.4" size="1.27" layer="96" display="off"/>
-<attribute name="MPN" x="10.16" y="25.4" size="1.27" layer="96" display="off"/>
-</instance>
-<instance part="H1" gate="G$1" x="10.16" y="33.02">
-<attribute name="OC_FARNELL" x="10.16" y="33.02" size="1.27" layer="96" display="off"/>
-<attribute name="MF" x="10.16" y="33.02" size="1.27" layer="96" display="off"/>
-<attribute name="MPN" x="10.16" y="33.02" size="1.27" layer="96" display="off"/>
+<instance part="H4" gate="G$1" x="17.78" y="10.16">
+<attribute name="OC_FARNELL" x="17.78" y="10.16" size="1.27" layer="96" display="off"/>
+<attribute name="MF" x="17.78" y="10.16" size="1.27" layer="96" display="off"/>
+<attribute name="MPN" x="17.78" y="10.16" size="1.27" layer="96" display="off"/>
+</instance>
+<instance part="H3" gate="G$1" x="17.78" y="17.78">
+<attribute name="OC_FARNELL" x="17.78" y="17.78" size="1.27" layer="96" display="off"/>
+<attribute name="MF" x="17.78" y="17.78" size="1.27" layer="96" display="off"/>
+<attribute name="MPN" x="17.78" y="17.78" size="1.27" layer="96" display="off"/>
+</instance>
+<instance part="H2" gate="G$1" x="17.78" y="25.4">
+<attribute name="OC_FARNELL" x="17.78" y="25.4" size="1.27" layer="96" display="off"/>
+<attribute name="MF" x="17.78" y="25.4" size="1.27" layer="96" display="off"/>
+<attribute name="MPN" x="17.78" y="25.4" size="1.27" layer="96" display="off"/>
+</instance>
+<instance part="H1" gate="G$1" x="17.78" y="33.02">
+<attribute name="OC_FARNELL" x="17.78" y="33.02" size="1.27" layer="96" display="off"/>
+<attribute name="MF" x="17.78" y="33.02" size="1.27" layer="96" display="off"/>
+<attribute name="MPN" x="17.78" y="33.02" size="1.27" layer="96" display="off"/>
 </instance>
 <instance part="S1" gate="BEF1" x="30.48" y="238.76">
@@
 <label x="152.4" y="193.04" size="1.27" layer="95" rot="R90" xref="yes"/>
 </segment>
+<segment>
+<pinref part="H1" gate="G$1" pin="MOUNT"/>
+<wire x1="15.24" y1="33.02" x2="12.7" y2="33.02" width="0.1524" layer="91"/>
+<label x="12.7" y="33.02" size="1.27" layer="95" rot="R180" xref="yes"/>
+</segment>
+<segment>
+<pinref part="H2" gate="G$1" pin="MOUNT"/>
+<wire x1="15.24" y1="25.4" x2="12.7" y2="25.4" width="0.1524" layer="91"/>
+<label x="12.7" y="25.4" size="1.27" layer="95" rot="R180" xref="yes"/>
+</segment>
+<segment>
+<wire x1="17.78" y1="17.78" x2="15.24" y2="17.78" width="0.1524" layer="91"/>
+<label x="12.7" y="17.78" size="1.27" layer="95" rot="R180" xref="yes"/>
+<pinref part="H3" gate="G$1" pin="MOUNT"/>
+<wire x1="15.24" y1="17.78" x2="12.7" y2="17.78" width="0.1524" layer="91"/>
+<junction x="15.24" y="17.78"/>
+</segment>
+<segment>
+<wire x1="17.78" y1="10.16" x2="15.24" y2="10.16" width="0.1524" layer="91"/>
+<label x="12.7" y="10.16" size="1.27" layer="95" rot="R180" xref="yes"/>
+<pinref part="H4" gate="G$1" pin="MOUNT"/>
+<wire x1="15.24" y1="10.16" x2="12.7" y2="10.16" width="0.1524" layer="91"/>
+<junction x="15.24" y="10.16"/>
+</segment>
 </net>
